File: ButtonHat/ButtonHat.sch (KiCad schematic (older format))
At the start: 36 parts, among them J0 RPI_GPIO, P1 CONN_6, P2 CONN_6, P3 CONN_6, P4 CONN_6, P5 CONN_6, P6 CONN_6, P7 CONN_2, U1 74AHC14, U2 74AHC14

Commit message: Final updates to schematic.
Parts:
- C7, C8: value 10 nf -> .1 uf
- J1: renamed from P2; value CONN_6 -> Buttons 1 to 6
- J2: renamed from P4; value CONN_6 -> Buttons 7 to 12
- J3: renamed from P5; value CONN_6 -> GPIO A
- J4: renamed from P6; value CONN_6 -> GPIO B
- T1: renamed from P1; value CONN_6 -> Buttons 1 to 6
- T2: renamed from P7; value CONN_2 -> Ground
- T3: renamed from P3; value CONN_6 -> Buttons 7 to 12

Commit message: Update GPIO Hats: make all 17 GPIO pins available on a socket header strip.
Parts:
- removed J3: GPIO A, ~, symbol CONN_6
- removed J4: GPIO B, ~, symbol CONN_6
- added J3: GPIO, ~, symbol CONN_17
Connections:
- net labels added: BCM12, wPi 26, BCM13, wPi 23, BCM16, wPi 27, BCM17, wPi 0, BCM18, wPi 1, BCM19, wPi 24, BCM20, wPi 28, BCM21, wPi 29, BCM22, wPi 3, BCM23, wPi 4, BCM24, wPi 5, BCM25, wPi 6, BCM26, wPi 25, BCM27, wPi 2, BCM4, wPi 7, BCM5, wPi 21, BCM6, wPi 22
- wire segments 118 -> 114
Changed lines of the file:
@@
 Sheet 1 1
 Title ""
-Date "2 oct 2017"
+Date "5 oct 2017"
 Rev ""
 Comp ""
@@
 $EndComp
 $Comp
-L CONN_6 J3
-U 1 1 59D27895
-P 7150 2450
-F 0 "J3" V 7100 2450 60  0000 C CNN
-F 1 "GPIO A" V 7200 2450 60  0000 C CNN
-F 2 "~" H 7150 2450 60  0000 C CNN
-F 3 "~" H 7150 2450 60  0000 C CNN
-	1    7150 2450
-	-1   0    0    -1
-$EndComp
-$Comp
-L CONN_6 J4
-U 1 1 59D278A4
-P 10600 2400
-F 0 "J4" V 10550 2400 60  0000 C CNN
-F 1 "GPIO B" V 10650 2400 60  0000 C CNN
-F 2 "~" H 10600 2400 60  0000 C CNN
-F 3 "~" H 10600 2400 60  0000 C CNN
-	1    10600 2400
-	1    0    0    -1
-$EndComp
-$Comp
 L +3.3V #PWR037
 U 1 1 59D28706
@@
 	1    2400 5450
 	1    0    0    -1
+$EndComp
+$Comp
+L CONN_2 T2
+U 1 1 59D28959
+P 1100 6550
+F 0 "T2" V 1050 6550 40  0000 C CNN
+F 1 "Ground" V 1150 6550 40  0000 C CNN
+F 2 "~" H 1100 6550 60  0000 C CNN
+F 3 "~" H 1100 6550 60  0000 C CNN
+	1    1100 6550
+	-1   0    0    -1
+$EndComp
+$Comp
+L GND #PWR041
+U 1 1 59D28968
+P 1450 6850
+F 0 "#PWR041" H 1450 6850 30  0001 C CNN
+F 1 "GND" H 1450 6780 30  0001 C CNN
+F 2 "" H 1450 6850 60  0000 C CNN
+F 3 "" H 1450 6850 60  0000 C CNN
+	1    1450 6850
+	1    0    0    -1
+$EndComp
+$Comp
+L CONN_17 J3
+U 1 1 59D63CAB
+P 9200 5150
+F 0 "J3" V 9160 5150 60  0000 C CNN
+F 1 "GPIO" V 9280 5150 60  0000 C CNN
+F 2 "~" H 9200 5150 60  0000 C CNN
+F 3 "~" H 9200 5150 60  0000 C CNN
+	1    9200 5150
+	0    -1   1    0
 $EndComp
 Wire Wire Line
@@
 	5850 5300 5700 5300
 Wire Wire Line
-	7950 1950 7500 1950
-Wire Wire Line
-	7500 1950 7500 2200
-Wire Wire Line
-	7950 2150 7950 2200
-Wire Wire Line
-	7950 2200 7550 2200
-Wire Wire Line
-	7550 2200 7550 2300
-Wire Wire Line
-	7550 2300 7500 2300
-Wire Wire Line
-	7950 2250 7600 2250
-Wire Wire Line
-	7600 2250 7600 2400
-Wire Wire Line
-	7600 2400 7500 2400
-Wire Wire Line
-	7950 2350 7700 2350
-Wire Wire Line
-	7700 2350 7700 2500
-Wire Wire Line
-	7700 2500 7500 2500
-Wire Wire Line
-	7950 3050 7650 3050
-Wire Wire Line
-	7650 3050 7650 2600
-Wire Wire Line
-	7650 2600 7500 2600
-Wire Wire Line
-	7950 3150 7500 3150
-Wire Wire Line
-	7500 3150 7500 2700
-Wire Wire Line
-	9850 2150 10250 2150
-Wire Wire Line
-	9850 2400 9850 2350
-Wire Wire Line
-	10250 2250 10000 2250
-Wire Wire Line
-	10000 2250 10000 2400
-Wire Wire Line
-	10000 2400 9850 2400
-Wire Wire Line
-	9850 2450 10050 2450
-Wire Wire Line
-	10050 2450 10050 2350
-Wire Wire Line
-	10050 2350 10250 2350
-Wire Wire Line
-	9850 2650 9850 2700
-Wire Wire Line
-	9850 2700 10100 2700
-Wire Wire Line
-	10100 2700 10100 2450
-Wire Wire Line
-	10100 2450 10250 2450
-Wire Wire Line
-	9850 3150 9850 3200
-Wire Wire Line
-	9850 3200 10150 3200
-Wire Wire Line
-	10150 3200 10150 2550
-Wire Wire Line
-	10150 2550 10250 2550
-Wire Wire Line
-	9850 3350 9850 3400
-Wire Wire Line
-	10250 3400 10250 2650
-Wire Wire Line
-	9850 3400 10250 3400
-Wire Wire Line
 	5200 5400 5200 5500
 Wire Wire Line
 	2400 5450 2400 5350
-$Comp
-L CONN_2 T2
-U 1 1 59D28959
-P 1100 6550
-F 0 "T2" V 1050 6550 40  0000 C CNN
-F 1 "Ground" V 1150 6550 40  0000 C CNN
-F 2 "~" H 1100 6550 60  0000 C CNN
-F 3 "~" H 1100 6550 60  0000 C CNN
-	1    1100 6550
-	-1   0    0    -1
-$EndComp
-$Comp
-L GND #PWR041
-U 1 1 59D28968
-P 1450 6850
-F 0 "#PWR041" H 1450 6850 30  0001 C CNN
-F 1 "GND" H 1450 6780 30  0001 C CNN
-F 2 "" H 1450 6850 60  0000 C CNN
-F 3 "" H 1450 6850 60  0000 C CNN
-	1    1450 6850
-	1    0    0    -1
-$EndComp
 Wire Wire Line
 	1450 6450 1450 6850
 Connection ~ 1450 6650
+Wire Wire Line
+	10050 2150 9850 2150
+Wire Wire Line
+	10050 2350 10000 2350
+Wire Wire Line
+	10000 2350 10000 2400
+Wire Wire Line
+	10000 2400 9850 2400
+Wire Wire Line
+	9850 2400 9850 2350
+Wire Wire Line
+	10050 2450 9850 2450
+Wire Wire Line
+	10050 2650 10000 2650
+Wire Wire Line
+	10000 2650 10000 2700
+Wire Wire Line
+	10000 2700 9850 2700
+Wire Wire Line
+	9850 2700 9850 2650
+Wire Wire Line
+	10050 3150 10000 3150
+Wire Wire Line
+	10000 3150 10000 3200
+Wire Wire Line
+	10000 3200 9850 3200
+Wire Wire Line
+	9850 3200 9850 3150
+Wire Wire Line
+	10050 3350 10000 3350
+Wire Wire Line
+	10000 3350 10000 3400
+Wire Wire Line
+	10000 3400 9850 3400
+Wire Wire Line
+	9850 3400 9850 3350
+Wire Wire Line
+	10050 3450 9850 3450
+Wire Wire Line
+	10050 3550 9850 3550
+Wire Wire Line
+	7700 1950 7950 1950
+Wire Wire Line
+	7700 2150 7750 2150
+Wire Wire Line
+	7750 2150 7750 2200
+Wire Wire Line
+	7750 2200 7950 2200
+Wire Wire Line
+	7950 2200 7950 2150
+Wire Wire Line
+	7700 2250 7950 2250
+Wire Wire Line
+	7700 2350 7950 2350
+Wire Wire Line
+	7700 3050 7950 3050
+Wire Wire Line
+	7700 3150 7950 3150
+Wire Wire Line
+	7700 3250 7950 3250
+Wire Wire Line
+	7700 3350 7950 3350
+Wire Wire Line
+	7700 3450 7950 3450
+Text GLabel 7700 1950 0    47   Input ~ 0
+BCM4, wPi 7
+Text GLabel 7700 2150 0    47   Input ~ 0
+BCM17, wPi 0
+Text GLabel 7700 2250 0    47   Input ~ 0
+BCM27, wPi 2
+Text GLabel 7700 2350 0    47   Input ~ 0
+BCM22, wPi 3
+Text GLabel 7700 3050 0    47   Input ~ 0
+BCM5, wPi 21
+Text GLabel 7700 3150 0    47   Input ~ 0
+BCM6, wPi 22
+Text GLabel 7700 3250 0    47   Input ~ 0
+BCM13, wPi 23
+Text GLabel 7700 3350 0    47   Input ~ 0
+BCM19, wPi 24
+Text GLabel 7700 3450 0    47   Input ~ 0
+BCM26, wPi 25
+Text GLabel 10050 2150 2    47   Input ~ 0
+BCM18, wPi 1
+Text GLabel 10050 2350 2    47   Input ~ 0
+BCM23, wPi 4
+Text GLabel 10050 2450 2    47   Input ~ 0
+BCM24, wPi 5
+Text GLabel 10050 2650 2    47   Input ~ 0
+BCM25, wPi 6
+Text GLabel 10050 3150 2    47   Input ~ 0
+BCM12, wPi 26
+Text GLabel 10050 3350 2    47   Input ~ 0
+BCM16, wPi 27
+Text GLabel 10050 3450 2    47   Input ~ 0
+BCM20, wPi 28
+Text GLabel 10050 3550 2    47   Input ~ 0
+BCM21, wPi 29
+Text GLabel 8400 4800 1    47   Input ~ 0
+BCM17, wPi 0
+Text GLabel 8500 4800 1    47   Input ~ 0
+BCM18, wPi 1
+Text GLabel 8600 4800 1    47   Input ~ 0
+BCM27, wPi 2
+Text GLabel 8700 4800 1    47   Input ~ 0
+BCM22, wPi 3
+Text GLabel 8800 4800 1    47   Input ~ 0
+BCM23, wPi 4
+Text GLabel 8900 4800 1    47   Input ~ 0
+BCM24, wPi 5
+Text GLabel 9000 4800 1    47   Input ~ 0
+BCM25, wPi 6
+Text GLabel 9100 4800 1    47   Input ~ 0
+BCM4, wPi 7
+Text GLabel 9200 4800 1    47   Input ~ 0
+BCM5, wPi 21
+Text GLabel 9300 4800 1    47   Input ~ 0
+BCM6, wPi 22
+Text GLabel 9400 4800 1    47   Input ~ 0
+BCM13, wPi 23
+Text GLabel 9500 4800 1    47   Input ~ 0
+BCM19, wPi 24
+Text GLabel 9600 4800 1    47   Input ~ 0
+BCM26, wPi 25
+Text GLabel 9700 4800 1    47   Input ~ 0
+BCM12, wPi 26
+Text GLabel 9800 4800 1    47   Input ~ 0
+BCM16, wPi 27
+Text GLabel 9900 4800 1    47   Input ~ 0
+BCM20, wPi 28
+Text GLabel 10000 4800 1    47   Input ~ 0
+BCM21, wPi 29
 $EndSCHEMATC

Commit message: Add BOM to ButtonHat.
Parts:
- C1, C10, C11, C12, C13, C14, C2, C3, C4, C5, C6, C9: Mouser Part Number (none) -> 21RZ410-RC
- C7, C8: Mouser Part Number (none) -> 21RZ310-RC
- J0: Adafruit  (none) -> 2223; Mouser Part Number (none) -> 855-M20-6102045
- J1, J2: Mouser Part Number (none) -> 538-90147-1106
- J3: Mouser Part Number (none) -> 517-929974-01-17-RK
- R1, R10, R11, R12, R2, R3, R4, R5, R6, R7, R8, R9: Mouser Part Number (none) -> 71-CCF5010K0FKE36
- T1, T3: Mouser Part Number (none) -> 651-1725698
- T2: Mouser Part Number (none) -> 571-282834-2
- U1, U2: Mouser Part Number (none) -> 595-SN74AHC14N
Changed lines of the file:
@@
 LIBS:microchip
 LIBS:analog_switches
-LIBS:74ahc14
 LIBS:motorola
 LIBS:texas
@@
 Sheet 1 1
 Title ""
-Date "5 oct 2017"
+Date "16 oct 2017"
 Rev ""
 Comp ""
@@
 F 2 "~" H 2450 1600 60  0000 C CNN
 F 3 "~" H 2450 1600 60  0000 C CNN
+F 4 "595-SN74AHC14N" H 2450 1600 60  0001 C CNN "Mouser Part Number"
 	1    2450 1600
 	1    0    0    -1
@@
 F 2 "~" H 5250 1650 60  0000 C CNN
 F 3 "~" H 5250 1650 60  0000 C CNN
+F 4 "595-SN74AHC14N" H 5250 1650 60  0001 C CNN "Mouser Part Number"
 	1    5250 1650
 	1    0    0    -1
@@
 F 2 "~" H 2038 1650 30  0000 C CNN
 F 3 "~" H 2000 1800 60  0000 C CNN
+F 4 "21RZ410-RC" H 2000 1800 60  0001 C CNN "Mouser Part Number"
 	1    2000 1800
 	1    0    0    -1
@@
 F 2 "~" H 2038 2350 30  0000 C CNN
 F 3 "~" H 2000 2500 60  0000 C CNN
+F 4 "21RZ410-RC" H 2000 1800 60  0001 C CNN "Mouser Part Number"
 	1    2000 2500
 	1    0    0    -1
@@
 F 2 "~" H 2038 3100 30  0000 C CNN
 F 3 "~" H 2000 3250 60  0000 C CNN
+F 4 "21RZ410-RC" H 2000 1800 60  0001 C CNN "Mouser Part Number"
 	1    2000 3250
 	1    0    0    -1
@@
 F 2 "~" H 2038 3850 30  0000 C CNN
 F 3 "~" H 2000 4000 60  0000 C CNN
+F 4 "21RZ410-RC" H 2000 1800 60  0001 C CNN "Mouser Part Number"
 	1    2000 4000
 	1    0    0    -1
@@
 F 2 "~" H 2038 4550 30  0000 C CNN
 F 3 "~" H 2000 4700 60  0000 C CNN
+F 4 "21RZ410-RC" H 2000 1800 60  0001 C CNN "Mouser Part Number"
 	1    2000 4700
 	1    0    0    -1
@@
 F 2 "~" H 2038 5300 30  0000 C CNN
 F 3 "~" H 2000 5450 60  0000 C CNN
+F 4 "21RZ410-RC" H 2000 1800 60  0001 C CNN "Mouser Part Number"
 	1    2000 5450
 	1    0    0    -1
@@
 F 2 "~" H 4838 5350 30  0000 C CNN
 F 3 "~" H 4800 5500 60  0000 C CNN
+F 4 "21RZ410-RC" H 2000 1800 60  0001 C CNN "Mouser Part Number"
 	1    4800 5500
 	1    0    0    -1
@@
 F 2 "~" H 4838 4600 30  0000 C CNN
 F 3 "~" H 4800 4750 60  0000 C CNN
+F 4 "21RZ410-RC" H 2000 1800 60  0001 C CNN "Mouser Part Number"
 	1    4800 4750
 	1    0    0    -1
@@
 F 2 "~" H 4838 3900 30  0000 C CNN
 F 3 "~" H 4800 4050 60  0000 C CNN
+F 4 "21RZ410-RC" H 2000 1800 60  0001 C CNN "Mouser Part Number"
 	1    4800 4050
 	1    0    0    -1
@@
 F 2 "~" H 4838 3150 30  0000 C CNN
 F 3 "~" H 4800 3300 60  0000 C CNN
+F 4 "21RZ410-RC" H 2000 1800 60  0001 C CNN "Mouser Part Number"
 	1    4800 3300
 	1    0    0    -1
@@
 F 2 "~" H 4838 2400 30  0000 C CNN
 F 3 "~" H 4800 2550 60  0000 C CNN
+F 4 "21RZ410-RC" H 2000 1800 60  0001 C CNN "Mouser Part Number"
 	1    4800 2550
 	1    0    0    -1
@@
 F 2 "~" H 4838 1700 30  0000 C CNN
 F 3 "~" H 4800 1850 60  0000 C CNN
+F 4 "21RZ410-RC" H 2000 1800 60  0001 C CNN "Mouser Part Number"
 	1    4800 1850
 	1    0    0    -1
@@
 F 2 "~" V 4530 1400 30  0000 C CNN
 F 3 "~" H 4600 1400 30  0000 C CNN
+F 4 "71-CCF5010K0FKE36" V 1800 1350 60  0001 C CNN "Mouser Part Number"
 	1    4600 1400
 	1    0    0    -1
@@
 F 2 "~" V 4530 2100 30  0000 C CNN
 F 3 "~" H 4600 2100 30  0000 C CNN
+F 4 "71-CCF5010K0FKE36" V 1800 1350 60  0001 C CNN "Mouser Part Number"
 	1    4600 2100
 	1    0    0    -1
@@
 F 2 "~" V 4530 2850 30  0000 C CNN
 F 3 "~" H 4600 2850 30  0000 C CNN
+F 4 "71-CCF5010K0FKE36" V 1800 1350 60  0001 C CNN "Mouser Part Number"
 	1    4600 2850
 	1    0    0    -1
@@
 F 2 "~" V 4530 3600 30  0000 C CNN
 F 3 "~" H 4600 3600 30  0000 C CNN
+F 4 "71-CCF5010K0FKE36" V 1800 1350 60  0001 C CNN "Mouser Part Number"
 	1    4600 3600
 	1    0    0    -1
@@
 F 2 "~" V 4530 4300 30  0000 C CNN
 F 3 "~" H 4600 4300 30  0000 C CNN
+F 4 "71-CCF5010K0FKE36" V 1800 1350 60  0001 C CNN "Mouser Part Number"
 	1    4600 4300
 	1    0    0    -1
@@
 F 2 "~" V 4530 5050 30  0000 C CNN
 F 3 "~" H 4600 5050 30  0000 C CNN
+F 4 "71-CCF5010K0FKE36" V 1800 1350 60  0001 C CNN "Mouser Part Number"
 	1    4600 5050
 	1    0    0    -1
@@
 F 2 "~" V 1730 1350 30  0000 C CNN
 F 3 "~" H 1800 1350 30  0000 C CNN
+F 4 "71-CCF5010K0FKE36" V 1800 1350 60  0001 C CNN "Mouser Part Number"
 	1    1800 1350
 	1    0    0    -1
@@
 F 2 "~" V 1730 2050 30  0000 C CNN
 F 3 "~" H 1800 2050 30  0000 C CNN
+F 4 "71-CCF5010K0FKE36" V 1800 1350 60  0001 C CNN "Mouser Part Number"
 	1    1800 2050
 	1    0    0    -1
@@
 F 2 "~" V 1730 2800 30  0000 C CNN
 F 3 "~" H 1800 2800 30  0000 C CNN
+F 4 "71-CCF5010K0FKE36" V 1800 1350 60  0001 C CNN "Mouser Part Number"
 	1    1800 2800
 	1    0    0    -1
@@
 F 2 "~" V 1730 3550 30  0000 C CNN
 F 3 "~" H 1800 3550 30  0000 C CNN
+F 4 "71-CCF5010K0FKE36" V 1800 1350 60  0001 C CNN "Mouser Part Number"
 	1    1800 3550
 	1    0    0    -1
@@
 F 2 "~" V 1730 4250 30  0000 C CNN
 F 3 "~" H 1800 4250 30  0000 C CNN
+F 4 "71-CCF5010K0FKE36" V 1800 1350 60  0001 C CNN "Mouser Part Number"
 	1    1800 4250
 	1    0    0    -1
@@
 F 2 "~" V 1730 5000 30  0000 C CNN
 F 3 "~" H 1800 5000 30  0000 C CNN
+F 4 "71-CCF5010K0FKE36" V 1800 1350 60  0001 C CNN "Mouser Part Number"
 	1    1800 5000
 	1    0    0    -1
@@
 F 2 "~" H 3888 6150 30  0000 C CNN
 F 3 "~" H 3850 6300 60  0000 C CNN
+F 4 "21RZ310-RC" H 3850 6300 60  0001 C CNN "Mouser Part Number"
 	1    3850 6300
 	1    0    0    -1
@@
 F 2 "~" H 3588 6150 30  0000 C CNN
 F 3 "~" H 3550 6300 60  0000 C CNN
+F 4 "21RZ310-RC" H 3550 6300 60  0001 C CNN "Mouser Part Number"
 	1    3550 6300
 	1    0    0    -1
@@
 F 2 "~" H 8150 1650 60  0000 C CNN
 F 3 "~" H 8150 1650 60  0000 C CNN
+F 4 "855-M20-6102045" H 1600 1450 60  0001 C CNN "Mouser Part Number"
+F 5 "2223" H 1600 1450 60  0001 C CNN "Adafruit "
 	1    8150 1650
 	1    0    0    -1
@@
 F 2 "~" H 800 3300 60  0000 C CNN
 F 3 "~" H 800 3300 60  0000 C CNN
+F 4 "651-1725698" V 800 3300 60  0001 C CNN "Mouser Part Number"
 	1    800  3300
 	-1   0    0    -1
@@
 F 2 "~" H 3400 3250 60  0000 C CNN
 F 3 "~" H 3400 3250 60  0000 C CNN
+F 4 "538-90147-1106" V 3400 3250 60  0001 C CNN "Mouser Part Number"
 	1    3400 3250
 	1    0    0    -1
@@
 F 2 "~" H 3750 3250 60  0000 C CNN
 F 3 "~" H 3750 3250 60  0000 C CNN
+F 4 "651-1725698" V 3750 3250 60  0001 C CNN "Mouser Part Number"
 	1    3750 3250
 	-1   0    0    -1
@@
 F 2 "~" H 6200 3250 60  0000 C CNN
 F 3 "~" H 6200 3250 60  0000 C CNN
+F 4 "538-90147-1106" V 6200 3250 60  0001 C CNN "Mouser Part Number"
 	1    6200 3250
 	1    0    0    -1
@@
 F 2 "~" H 1100 6550 60  0000 C CNN
 F 3 "~" H 1100 6550 60  0000 C CNN
+F 4 "571-282834-2" V 8150 1300 60  0001 C CNN "Mouser Part Number"
 	1    1100 6550
 	-1   0    0    -1
@@
 F 2 "~" H 9200 5150 60  0000 C CNN
 F 3 "~" H 9200 5150 60  0000 C CNN
+F 4 "517-929974-01-17-RK" V 8100 6100 60  0001 C CNN "Mouser Part Number"
 	1    9200 5150
 	0    -1   1    0

Commit message: Update 10nf caps to a stocked Mouser part.
Parts:
- C1, C10, C11, C12, C13, C14, C2, C3, C4, C5, C6, C9: Mouser Part Number 21RZ410-RC -> 80-C317C103M5U
Changed lines of the file:
@@
 F 2 "~" H 2038 1650 30  0000 C CNN
 F 3 "~" H 2000 1800 60  0000 C CNN
-F 4 "21RZ410-RC" H 2000 1800 60  0001 C CNN "Mouser Part Number"
+F 4 "80-C317C103M5U" H 2000 1800 60  0001 C CNN "Mouser Part Number"
 	1    2000 1800
 	1    0    0    -1
@@
 F 2 "~" H 2038 2350 30  0000 C CNN
 F 3 "~" H 2000 2500 60  0000 C CNN
-F 4 "21RZ410-RC" H 2000 1800 60  0001 C CNN "Mouser Part Number"
+F 4 "80-C317C103M5U" H 2000 1800 60  0001 C CNN "Mouser Part Number"
 	1    2000 2500
 	1    0    0    -1
@@
 F 2 "~" H 2038 3100 30  0000 C CNN
 F 3 "~" H 2000 3250 60  0000 C CNN
-F 4 "21RZ410-RC" H 2000 1800 60  0001 C CNN "Mouser Part Number"
+F 4 "80-C317C103M5U" H 2000 1800 60  0001 C CNN "Mouser Part Number"
 	1    2000 3250
 	1    0    0    -1
@@
 F 2 "~" H 2038 3850 30  0000 C CNN
 F 3 "~" H 2000 4000 60  0000 C CNN
-F 4 "21RZ410-RC" H 2000 1800 60  0001 C CNN "Mouser Part Number"
+F 4 "80-C317C103M5U" H 2000 1800 60  0001 C CNN "Mouser Part Number"
 	1    2000 4000
 	1    0    0    -1
@@
 F 2 "~" H 2038 4550 30  0000 C CNN
 F 3 "~" H 2000 4700 60  0000 C CNN
-F 4 "21RZ410-RC" H 2000 1800 60  0001 C CNN "Mouser Part Number"
+F 4 "80-C317C103M5U" H 2000 1800 60  0001 C CNN "Mouser Part Number"
 	1    2000 4700
 	1    0    0    -1
@@
 F 2 "~" H 2038 5300 30  0000 C CNN
 F 3 "~" H 2000 5450 60  0000 C CNN
-F 4 "21RZ410-RC" H 2000 1800 60  0001 C CNN "Mouser Part Number"
+F 4 "80-C317C103M5U" H 2000 1800 60  0001 C CNN "Mouser Part Number"
 	1    2000 5450
 	1    0    0    -1
@@
 F 2 "~" H 4838 5350 30  0000 C CNN
 F 3 "~" H 4800 5500 60  0000 C CNN
-F 4 "21RZ410-RC" H 2000 1800 60  0001 C CNN "Mouser Part Number"
+F 4 "80-C317C103M5U" H 2000 1800 60  0001 C CNN "Mouser Part Number"
 	1    4800 5500
 	1    0    0    -1
@@
 F 2 "~" H 4838 4600 30  0000 C CNN
 F 3 "~" H 4800 4750 60  0000 C CNN
-F 4 "21RZ410-RC" H 2000 1800 60  0001 C CNN "Mouser Part Number"
+F 4 "80-C317C103M5U" H 2000 1800 60  0001 C CNN "Mouser Part Number"
 	1    4800 4750
 	1    0    0    -1
@@
 F 2 "~" H 4838 3900 30  0000 C CNN
 F 3 "~" H 4800 4050 60  0000 C CNN
-F 4 "21RZ410-RC" H 2000 1800 60  0001 C CNN "Mouser Part Number"
+F 4 "80-C317C103M5U" H 2000 1800 60  0001 C CNN "Mouser Part Number"
 	1    4800 4050
 	1    0    0    -1
@@
 F 2 "~" H 4838 3150 30  0000 C CNN
 F 3 "~" H 4800 3300 60  0000 C CNN
-F 4 "21RZ410-RC" H 2000 1800 60  0001 C CNN "Mouser Part Number"
+F 4 "80-C317C103M5U" H 2000 1800 60  0001 C CNN "Mouser Part Number"
 	1    4800 3300
 	1    0    0    -1
@@
 F 2 "~" H 4838 2400 30  0000 C CNN
 F 3 "~" H 4800 2550 60  0000 C CNN
-F 4 "21RZ410-RC" H 2000 1800 60  0001 C CNN "Mouser Part Number"
+F 4 "80-C317C103M5U" H 2000 1800 60  0001 C CNN "Mouser Part Number"
 	1    4800 2550
 	1    0    0    -1
@@
 F 2 "~" H 4838 1700 30  0000 C CNN
 F 3 "~" H 4800 1850 60  0000 C CNN
-F 4 "21RZ410-RC" H 2000 1800 60  0001 C CNN "Mouser Part Number"
+F 4 "80-C317C103M5U" H 2000 1800 60  0001 C CNN "Mouser Part Number"
 	1    4800 1850
 	1    0    0    -1
