File: DCCTiva/DCCTiva.sch (KiCad schematic (older format))
At the start: 11 parts, among them J1 TI_BOOSTER_40_J1, J2 TI_BOOSTER_40_J2, J3 TI_BOOSTER_40_J3, J4 TI_BOOSTER_40_J4, J5 CONN_3

Commit message: Finalize the circuit
Parts:
- added P1: Power and DCC, ~, symbol CONN_4
- gave numbers to parts that had none: 6
Connections:
- net labels added: DCC A, DCC B
Changed lines of the file:
@@
 $EndComp
 $Comp
-L LMD18200 U?
+L LMD18200 U1
 U 1 1 5A7B1E9B
 P 7050 1200
-F 0 "U?" H 7050 1200 60  0000 C CNN
+F 0 "U1" H 7050 1200 60  0000 C CNN
 F 1 "LMD18200" H 7050 1300 60  0000 C CNN
 F 2 "~" H 7050 1200 60  0000 C CNN
@@
 $EndComp
 $Comp
-L C C?
+L C C2
 U 1 1 5A7B1EAA
 P 7500 1700
-F 0 "C?" H 7500 1800 40  0000 L CNN
+F 0 "C2" H 7500 1800 40  0000 L CNN
 F 1 ".01 uf" H 7506 1615 40  0000 L CNN
 F 2 "~" H 7538 1550 30  0000 C CNN
@@
 $EndComp
 $Comp
-L C C?
+L C C1
 U 1 1 5A7B1EB9
 P 6600 1700
-F 0 "C?" H 6600 1800 40  0000 L CNN
+F 0 "C1" H 6600 1800 40  0000 L CNN
 F 1 ".01 uf" H 6606 1615 40  0000 L CNN
 F 2 "~" H 6638 1550 30  0000 C CNN
@@
 $EndComp
 $Comp
-L R R?
+L R R1
 U 1 1 5A7B1EC8
 P 7150 1900
-F 0 "R?" V 7230 1900 40  0000 C CNN
+F 0 "R1" V 7230 1900 40  0000 C CNN
 F 1 "2.7K Ohms" V 7157 1901 40  0000 C CNN
 F 2 "~" V 7080 1900 30  0000 C CNN
@@
 $EndComp
 $Comp
-L R R?
+L R R2
 U 1 1 5A7B1ED7
 P 8100 1300
-F 0 "R?" V 8180 1300 40  0000 C CNN
+F 0 "R2" V 8180 1300 40  0000 C CNN
 F 1 "2.7K Ohms" V 8107 1301 40  0000 C CNN
 F 2 "~" V 8030 1300 30  0000 C CNN
@@
 $EndComp
 $Comp
-L LED D?
+L LED D1
 U 1 1 5A7B1EE6
 P 8100 850
-F 0 "D?" H 8100 950 50  0000 C CNN
+F 0 "D1" H 8100 950 50  0000 C CNN
 F 1 "Thermal Warning" H 8100 750 50  0000 C CNN
 F 2 "~" H 8100 850 60  0000 C CNN
@@
 	7250 1900 7500 1900
 $Comp
-L VCC #PWR?
+L VCC #PWR07
 U 1 1 5A7B1FB5
 P 7000 1500
-F 0 "#PWR?" H 7000 1600 30  0001 C CNN
+F 0 "#PWR07" H 7000 1600 30  0001 C CNN
 F 1 "VCC" H 7000 1600 30  0000 C CNN
 F 2 "" H 7000 1500 60  0000 C CNN
@@
 	7050 2150 7150 2150
 $Comp
-L GND #PWR?
+L GND #PWR08
 U 1 1 5A7B2030
 P 7150 2250
-F 0 "#PWR?" H 7150 2250 30  0001 C CNN
+F 0 "#PWR08" H 7150 2250 30  0001 C CNN
 F 1 "GND" H 7150 2180 30  0001 C CNN
 F 2 "" H 7150 2250 60  0000 C CNN
@@
 	7200 1550 7200 1500
 $Comp
-L +5V #PWR?
+L +5V #PWR09
 U 1 1 5A7B20C2
 P 8100 650
-F 0 "#PWR?" H 8100 740 20  0001 C CNN
+F 0 "#PWR09" H 8100 740 20  0001 C CNN
 F 1 "+5V" H 8100 740 30  0000 C CNN
 F 2 "" H 8100 650 60  0000 C CNN
@@
 Wire Wire Line
 	6900 2100 6900 1500
+Text Label 9150 4800 2    60   ~ 0
+Current Sense
+Text Label 6600 1900 2    60   ~ 0
+DCC A
+Text Label 7500 1900 0    60   ~ 0
+DCC B
+$Comp
+L CONN_4 P1
+U 1 1 5A7B253F
+P 7550 2850
+F 0 "P1" V 7500 2850 50  0000 C CNN
+F 1 "Power and DCC" V 7600 2850 50  0000 C CNN
+F 2 "~" H 7550 2850 60  0000 C CNN
+F 3 "~" H 7550 2850 60  0000 C CNN
+	1    7550 2850
+	1    0    0    -1
+$EndComp
+Text Label 7200 2700 2    60   ~ 0
++15V
+$Comp
+L GND #PWR010
+U 1 1 5A7B2563
+P 7200 2800
+F 0 "#PWR010" H 7200 2800 30  0001 C CNN
+F 1 "GND" H 7200 2730 30  0001 C CNN
+F 2 "" H 7200 2800 60  0000 C CNN
+F 3 "" H 7200 2800 60  0000 C CNN
+	1    7200 2800
+	0    1    1    0
+$EndComp
+Text Label 7200 2900 2    60   ~ 0
+DCC A
+Text Label 7200 3000 2    60   ~ 0
+DCC B
 $EndSCHEMATC

Commit message: Add support for I2C LCD.
Parts:
- added P2: I2C 1, ~, symbol CONN_4
- added P3: I2C 0, ~, symbol CONN_4
Connections:
- net labels added: SCL - 0, SCL - 1, SDA - 0, SDA - 1
Changed lines of the file:
@@
 Sheet 1 1
 Title ""
-Date "7 feb 2018"
+Date "10 feb 2018"
 Rev ""
 Comp ""
@@
 Text Label 7200 3000 2    60   ~ 0
 DCC B
+$Comp
+L CONN_4 P2
+U 1 1 5A7F8158
+P 7450 3500
+F 0 "P2" V 7400 3500 50  0000 C CNN
+F 1 "I2C 1" V 7500 3500 50  0000 C CNN
+F 2 "~" H 7450 3500 60  0000 C CNN
+F 3 "~" H 7450 3500 60  0000 C CNN
+	1    7450 3500
+	-1   0    0    -1
+$EndComp
+$Comp
+L GND #PWR011
+U 1 1 5A7F81A1
+P 7800 3350
+F 0 "#PWR011" H 7800 3350 30  0001 C CNN
+F 1 "GND" H 7800 3280 30  0001 C CNN
+F 2 "" H 7800 3350 60  0000 C CNN
+F 3 "" H 7800 3350 60  0000 C CNN
+	1    7800 3350
+	0    -1   -1   0
+$EndComp
+$Comp
+L +5V #PWR012
+U 1 1 5A7F81B0
+P 7800 3450
+F 0 "#PWR012" H 7800 3540 20  0001 C CNN
+F 1 "+5V" H 7800 3540 30  0000 C CNN
+F 2 "" H 7800 3450 60  0000 C CNN
+F 3 "" H 7800 3450 60  0000 C CNN
+	1    7800 3450
+	0    1    1    0
+$EndComp
+Text Label 7800 3550 0    60   ~ 0
+SDA - 1
+Text Label 7800 3650 0    60   ~ 0
+SCL - 1
+Text Label 9150 1700 2    60   ~ 0
+SCL - 1
+Text Label 9150 1800 2    60   ~ 0
+SDA - 1
+Text Label 9150 2550 2    60   ~ 0
+SCL - 0
+Text Label 9150 5750 2    60   ~ 0
+SDA - 0
+$Comp
+L CONN_4 P3
+U 1 1 5A7F86EA
+P 7450 4000
+F 0 "P3" V 7400 4000 50  0000 C CNN
+F 1 "I2C 0" V 7500 4000 50  0000 C CNN
+F 2 "~" H 7450 4000 60  0000 C CNN
+F 3 "~" H 7450 4000 60  0000 C CNN
+	1    7450 4000
+	-1   0    0    -1
+$EndComp
+$Comp
+L GND #PWR013
+U 1 1 5A7F871E
+P 7800 3850
+F 0 "#PWR013" H 7800 3850 30  0001 C CNN
+F 1 "GND" H 7800 3780 30  0001 C CNN
+F 2 "" H 7800 3850 60  0000 C CNN
+F 3 "" H 7800 3850 60  0000 C CNN
+	1    7800 3850
+	0    -1   -1   0
+$EndComp
+$Comp
+L +5V #PWR014
+U 1 1 5A7F8732
+P 7800 3950
+F 0 "#PWR014" H 7800 4040 20  0001 C CNN
+F 1 "+5V" H 7800 4040 30  0000 C CNN
+F 2 "" H 7800 3950 60  0000 C CNN
+F 3 "" H 7800 3950 60  0000 C CNN
+	1    7800 3950
+	0    1    1    0
+$EndComp
+Text Label 7800 4050 0    60   ~ 0
+SDA - 0
+Text Label 7800 4150 0    60   ~ 0
+SCL - 0
 $EndSCHEMATC
