File: DCCOD_SMD/DCCOD_SMD.sch (KiCad schematic (older format))
At the start: 27 parts, among them P1 10K Ohms, P101 CONN_2, P102 CONN_4, Q1 CMUT3904, U1 LM324

Commit message: Change pot to side addjust (upright)
Parts:
- P1: Mouser Part Number 652-TC33X-2-103E -> 652-3313S-1-103E
Connections:
- net labels added: +5V
- net labels removed: +12V
Changed lines of the file:
@@
 Sheet 1 1
 Title ""
-Date "12 nov 2019"
+Date "14 nov 2019"
 Rev ""
 Comp ""
@@
 $EndComp
 $Comp
-L +12V #PWR01
+L +5V #PWR01
 U 1 1 5DCAB110
 P 1250 2100
 F 0 "#PWR01" H 1250 2050 20  0001 C CNN
-F 1 "+12V" H 1250 2200 30  0000 C CNN
+F 1 "+5V" H 1250 2200 30  0000 C CNN
 F 2 "" H 1250 2100 60  0000 C CNN
 F 3 "" H 1250 2100 60  0000 C CNN
@@
 Connection ~ 2850 2900
 $Comp
-L +12V #PWR03
+L +5V #PWR03
 U 1 1 5DCAB362
 P 2850 2200
 F 0 "#PWR03" H 2850 2150 20  0001 C CNN
-F 1 "+12V" H 2850 2300 30  0000 C CNN
+F 1 "+5V" H 2850 2300 30  0000 C CNN
 F 2 "" H 2850 2200 60  0000 C CNN
 F 3 "" H 2850 2200 60  0000 C CNN
@@
 	4650 3550 4650 3000
 $Comp
-L +12V #PWR05
+L +5V #PWR05
 U 1 1 5DCAB4EB
 P 4050 2400
 F 0 "#PWR05" H 4050 2350 20  0001 C CNN
-F 1 "+12V" H 4050 2500 30  0000 C CNN
+F 1 "+5V" H 4050 2500 30  0000 C CNN
 F 2 "" H 4050 2400 60  0000 C CNN
 F 3 "" H 4050 2400 60  0000 C CNN
@@
 F 2 "~" H 5550 3100 60  0000 C CNN
 F 3 "~" H 5550 3100 60  0000 C CNN
-F 4 "652-TC33X-2-103E" H 5550 3100 60  0001 C CNN "Mouser Part Number"
+F 4 "652-3313S-1-103E" H 5550 3100 60  0001 C CNN "Mouser Part Number"
 	1    5550 3100
 	0    1    -1   0
@@
 Connection ~ 5550 2800
 $Comp
-L +12V #PWR08
+L +5V #PWR08
 U 1 1 5DCAB7CF
 P 5550 2050
 F 0 "#PWR08" H 5550 2000 20  0001 C CNN
-F 1 "+12V" H 5550 2150 30  0000 C CNN
+F 1 "+5V" H 5550 2150 30  0000 C CNN
 F 2 "" H 5550 2050 60  0000 C CNN
 F 3 "" H 5550 2050 60  0000 C CNN
@@
 	6800 2200 6800 2300
 $Comp
-L +12V #PWR09
+L +5V #PWR09
 U 1 1 5DCAB886
 P 6800 1650
 F 0 "#PWR09" H 6800 1600 20  0001 C CNN
-F 1 "+12V" H 6800 1750 30  0000 C CNN
+F 1 "+5V" H 6800 1750 30  0000 C CNN
 F 2 "" H 6800 1650 60  0000 C CNN
 F 3 "" H 6800 1650 60  0000 C CNN
@@
 Connection ~ 8400 2700
 $Comp
-L +12V #PWR011
+L +5V #PWR011
 U 1 1 5DCABBDC
 P 8400 2000
 F 0 "#PWR011" H 8400 1950 20  0001 C CNN
-F 1 "+12V" H 8400 2100 30  0000 C CNN
+F 1 "+5V" H 8400 2100 30  0000 C CNN
 F 2 "" H 8400 2000 60  0000 C CNN
 F 3 "" H 8400 2000 60  0000 C CNN
@@
 $EndComp
 $Comp
-L +12V #PWR015
+L +5V #PWR015
 U 1 1 5DCB07CB
 P 10700 1950
 F 0 "#PWR015" H 10700 1900 20  0001 C CNN
-F 1 "+12V" H 10700 2050 30  0000 C CNN
+F 1 "+5V" H 10700 2050 30  0000 C CNN
 F 2 "" H 10700 1950 60  0000 C CNN
 F 3 "" H 10700 1950 60  0000 C CNN
