File: ESP32-16PWMLedDriver/PCA9685Driver.sch (KiCad schematic (older format))
At the start: 18 parts, among them P401 C A0 A1 A2 A3 A4 A5 A6 A7, P402 C B0 B1 B2 B3 B4 B5 B6 B7, T401 + 12V -, U401 PCA9685, U402 TBD62X83A, U403 TBD62X83A

Commit message: ESP32-16PWMLedDriver updates
Parts:
- C401: symbol C -> C-RESCUE-ESP32-16PWMLedDriver
Changed lines of the file:
@@
 EESchema Schematic File Version 2
+LIBS:ESP32-16PWMLedDriver-rescue
 LIBS:power
 LIBS:device
@@
 LIBS:memory
 LIBS:xilinx
-LIBS:special
 LIBS:microcontrollers
 LIBS:dsp
@@
 LIBS:pca9685
 LIBS:ESP32-16PWMLedDriver-cache
-EELAYER 27 0
+EELAYER 25 0
 EELAYER END
 $Descr A4 11693 8268
@@
 $EndComp
 $Comp
-L GND #PWR014
+L GND-RESCUE-ESP32-16PWMLedDriver #PWR014
 U 1 1 5E334BBC
 P 2800 3050
@@
 $EndComp
 $Comp
-L C C401
+L C-RESCUE-ESP32-16PWMLedDriver C401
 U 1 1 5E334BBD
 P 3550 1600
@@
 $EndComp
 $Comp
-L GND #PWR015
+L GND-RESCUE-ESP32-16PWMLedDriver #PWR015
 U 1 1 5E334BBE
 P 3550 1850
@@
 $EndComp
 $Comp
-L GND #PWR020
+L GND-RESCUE-ESP32-16PWMLedDriver #PWR020
 U 1 1 5E334BDB
 P 4550 5350
@@
 $EndComp
 $Comp
-L GND #PWR021
+L GND-RESCUE-ESP32-16PWMLedDriver #PWR021
 U 1 1 5E334BDC
 P 7050 5300
@@
 $EndComp
 $Comp
-L GND #PWR022
+L GND-RESCUE-ESP32-16PWMLedDriver #PWR022
 U 1 1 5E334BDD
 P 7550 750
@@
 $EndComp
 $Comp
-L GND #PWR023
+L GND-RESCUE-ESP32-16PWMLedDriver #PWR023
 U 1 1 5E334BDE
 P 5050 750
@@
 $EndComp
 $Comp
-L GND #PWR024
+L GND-RESCUE-ESP32-16PWMLedDriver #PWR024
 U 1 1 5E334BE0
 P 1200 3100
@@
 	2850 5050 3300 5050
 $Comp
-L GND #PWR026
+L GND-RESCUE-ESP32-16PWMLedDriver #PWR026
 U 1 1 5E334F18
 P 2850 5350
