File: ESP32-16xDCCOD/ESP32-16xDCCOD.sch (KiCad schematic (older format))
At the start: 20 parts, among them P101 CONN_4, P102 CONN_4, P103 CONN_4, P104 CONN_4, P105 CONN_4, P106 CONN_4, P107 CONN_4, P108 CONN_4, P109 CONN_4, P110 CONN_4, P111 CONN_4, P112 CONN_4, P113 CONN_4, P114 CONN_4, P115 CONN_4, P116 CONN_4, U0 ESP32_DEVKIT_C or TTGO-T1, U101 MCP23017

Commit message: Working on PocketBeagleCommandStation
Parts:
- C101: symbol C -> C-RESCUE-ESP32-16xDCCOD
- R101: symbol R -> R-RESCUE-ESP32-16xDCCOD
- U101: symbol MCP23017 -> MCP23017-RESCUE-ESP32-16xDCCOD
Changed lines of the file:
@@
 EESchema Schematic File Version 2
+LIBS:ESP32-16xDCCOD-rescue
 LIBS:power
 LIBS:device
@@
 LIBS:memory
 LIBS:xilinx
-LIBS:special
 LIBS:microcontrollers
 LIBS:dsp
@@
 LIBS:MCP23xxx
 LIBS:ESP32-16xDCCOD-cache
-EELAYER 27 0
+EELAYER 25 0
 EELAYER END
 $Descr A4 11693 8268
@@
 $EndComp
 $Comp
-L GND #PWR01
+L GND-RESCUE-ESP32-16xDCCOD #PWR01
 U 1 1 5C81D000
 P 2500 2200
@@
 $EndComp
 $Comp
-L GND #PWR03
+L GND-RESCUE-ESP32-16xDCCOD #PWR03
 U 1 1 5C81D02F
 P 3700 1550
@@
 $EndSheet
 $Comp
-L MCP23017 U101
+L MCP23017-RESCUE-ESP32-16xDCCOD U101
 U 1 1 5DCD62E1
 P 6150 3950
@@
 $EndComp
 $Comp
-L GND #PWR06
+L GND-RESCUE-ESP32-16xDCCOD #PWR06
 U 1 1 5DCD750E
 P 7350 4100
@@
 $EndComp
 $Comp
-L R R101
+L R-RESCUE-ESP32-16xDCCOD R101
 U 1 1 5DCD76F9
 P 5300 3250
@@
 Connection ~ 7100 5900
 $Comp
-L GND #PWR08
+L GND-RESCUE-ESP32-16xDCCOD #PWR08
 U 1 1 5DCDA08A
 P 7550 5900
@@
 OD2
 $Comp
-L C C101
+L C-RESCUE-ESP32-16xDCCOD C101
 U 1 1 5DCDBFFB
 P 4900 4150
