File: ESP32-16xDCCOD/PowerSupply.sch (KiCad schematic (older format))
At the start: 5 parts, among them U3 LM2574N-5.0

Commit message: Working on PocketBeagleCommandStation
Parts:
- C4, C5: symbol CP1 -> CP1-RESCUE-ESP32-16xDCCOD
Changed lines of the file:
@@
 EESchema Schematic File Version 2
+LIBS:ESP32-16xDCCOD-rescue
 LIBS:power
 LIBS:device
@@
 LIBS:memory
 LIBS:xilinx
-LIBS:special
 LIBS:microcontrollers
 LIBS:dsp
@@
 LIBS:MCP23xxx
 LIBS:ESP32-16xDCCOD-cache
-EELAYER 27 0
+EELAYER 25 0
 EELAYER END
 $Descr A4 11693 8268
@@
 $EndComp
 $Comp
-L CP1 C5
+L CP1-RESCUE-ESP32-16xDCCOD C5
 U 1 1 5C829D01
 P 5950 2900
@@
 $EndComp
 $Comp
-L CP1 C4
+L CP1-RESCUE-ESP32-16xDCCOD C4
 U 1 1 5C829D34
 P 3700 2800
@@
 Connection ~ 4850 3300
 $Comp
-L GND #PWR017
+L GND-RESCUE-ESP32-16xDCCOD #PWR017
 U 1 1 5C829DEF
 P 4850 3400
