File: ESP32-PWMHalfSidingSMD/PowerSupply.sch (KiCad schematic (older format))
At the start: 5 parts, among them U3 LM2574N-5.0

Commit message: Restore PocketBeagleCommandStation_SMD.kicad_pcb
Parts:
- C4, C5: footprint Capacitors_SMD:CP_Elec_8x10 -> ~; symbol CP1-RESCUE-ESP32-PWMHalfSidingSMD -> CP1
- D3: footprint Diodes_SMD:D_SMB -> ~
- L1: footprint SRN1060:SRN1060 -> ~
- U3: footprint SOIC_Wide:SOIC-14_7.4x8.7mm_Pitch1.27mm -> ~
Changed lines of the file:
@@
 EESchema Schematic File Version 2
-LIBS:ESP32-PWMHalfSidingSMD-rescue
 LIBS:power
 LIBS:device
@@
 LIBS:memory
 LIBS:xilinx
+LIBS:special
 LIBS:microcontrollers
 LIBS:dsp
@@
 LIBS:4814p-2
 LIBS:ESP32-PWMHalfSidingSMD-cache
-EELAYER 25 0
+EELAYER 27 0
 EELAYER END
 $Descr A4 11693 8268
@@
 F 0 "U3" H 5200 2850 60  0000 C CNN
 F 1 "LM2574N-5.0" H 5200 2950 21  0000 C CNN
-F 2 "SOIC_Wide:SOIC-14_7.4x8.7mm_Pitch1.27mm" H 5200 2800 60  0001 C CNN
+F 2 "~" H 5200 2800 60  0000 C CNN
 F 3 "~" H 5200 2800 60  0000 C CNN
 F 4 "926-LM2574N-5.0/NOPB" H 5200 2800 60  0001 C CNN "Mouser Part Number"
@@
 $EndComp
 $Comp
-L CP1-RESCUE-ESP32-PWMHalfSidingSMD C5
+L CP1 C5
 U 1 1 5C829D01
 P 5950 2900
 F 0 "C5" H 6000 3000 50  0000 L CNN
 F 1 "22 uf 100V" H 6000 2800 50  0000 L CNN
-F 2 "Capacitors_SMD:CP_Elec_8x10" H 5950 2900 60  0001 C CNN
+F 2 "~" H 5950 2900 60  0000 C CNN
 F 3 "~" H 5950 2900 60  0000 C CNN
 F 4 "647-UUX2A220MNL6GS" H 5950 2900 60  0001 C CNN "Mouser Part Number"
@@
 $EndComp
 $Comp
-L CP1-RESCUE-ESP32-PWMHalfSidingSMD C4
+L CP1 C4
 U 1 1 5C829D34
 P 3700 2800
 F 0 "C4" H 3750 2900 50  0000 L CNN
 F 1 "220 uf 25V" H 3750 2700 50  0000 L CNN
-F 2 "Capacitors_SMD:CP_Elec_8x10" H 3700 2800 60  0001 C CNN
+F 2 "~" H 3700 2800 60  0000 C CNN
 F 3 "~" H 3700 2800 60  0000 C CNN
 F 4 "647-UWT1E221MNL1GS" H 3700 2800 60  0001 C CNN "Mouser Part Number"
@@
 F 0 "L1" H 4550 3000 50  0000 C CNN
 F 1 "330 uh" H 4550 2850 50  0000 C CNN
-F 2 "SRN1060:SRN1060" H 4550 2900 60  0001 C CNN
+F 2 "~" H 4550 2900 60  0000 C CNN
 F 3 "~" H 4550 2900 60  0000 C CNN
 F 4 "652-SRN1060-331M" H 4550 2900 60  0001 C CNN "Mouser Part Number"
@@
 F 0 "D3" H 4850 3200 40  0000 C CNN
 F 1 "CMSH1-60 TR13" H 4850 3000 40  0000 C CNN
-F 2 "Diodes_SMD:D_SMB" H 4850 3100 60  0001 C CNN
+F 2 "~" H 4850 3100 60  0000 C CNN
 F 3 "~" H 4850 3100 60  0000 C CNN
 F 4 "610-CMSH1-60TR13" H 4850 3100 60  0001 C CNN "Mouser Part Number"
@@
 Connection ~ 4850 3300
 $Comp
-L GND-RESCUE-ESP32-PWMHalfSidingSMD #PWR015
+L GND #PWR015
 U 1 1 5C829DEF
 P 4850 3400
@@
 Wire Wire Line
 	4850 3300 4850 3400
-Text GLabel 5950 2550 2    100  Input ~ 0
+Text GLabel 5950 2550 0    100  Input ~ 0
 CAN +12V
 $EndSCHEMATC

Commit message: Repair ESP32-PWMHalfSidingSMD and generate POS file.
Parts:
- C4, C5: footprint ~ -> Capacitors_SMD:CP_Elec_8x10; symbol CP1 -> CP1-RESCUE-ESP32-PWMHalfSidingSMD
- D3: footprint ~ -> Diodes_SMD:D_SMB
- L1: footprint ~ -> SRN1060:SRN1060
- U3: footprint ~ -> (none)
Changed lines of the file:
@@
 EESchema Schematic File Version 2
+LIBS:ESP32-PWMHalfSidingSMD-rescue
 LIBS:power
 LIBS:device
@@
 LIBS:memory
 LIBS:xilinx
-LIBS:special
 LIBS:microcontrollers
 LIBS:dsp
@@
 LIBS:4814p-2
 LIBS:ESP32-PWMHalfSidingSMD-cache
-EELAYER 27 0
+EELAYER 25 0
 EELAYER END
 $Descr A4 11693 8268
@@
 F 0 "U3" H 5200 2850 60  0000 C CNN
 F 1 "LM2574N-5.0" H 5200 2950 21  0000 C CNN
-F 2 "~" H 5200 2800 60  0000 C CNN
+F 2 "" H 5200 2800 60  0001 C CNN
 F 3 "~" H 5200 2800 60  0000 C CNN
 F 4 "926-LM2574N-5.0/NOPB" H 5200 2800 60  0001 C CNN "Mouser Part Number"
@@
 $EndComp
 $Comp
-L CP1 C5
+L CP1-RESCUE-ESP32-PWMHalfSidingSMD C5
 U 1 1 5C829D01
 P 5950 2900
 F 0 "C5" H 6000 3000 50  0000 L CNN
 F 1 "22 uf 100V" H 6000 2800 50  0000 L CNN
-F 2 "~" H 5950 2900 60  0000 C CNN
+F 2 "Capacitors_SMD:CP_Elec_8x10" H 5950 2900 60  0001 C CNN
 F 3 "~" H 5950 2900 60  0000 C CNN
 F 4 "647-UUX2A220MNL6GS" H 5950 2900 60  0001 C CNN "Mouser Part Number"
@@
 $EndComp
 $Comp
-L CP1 C4
+L CP1-RESCUE-ESP32-PWMHalfSidingSMD C4
 U 1 1 5C829D34
 P 3700 2800
 F 0 "C4" H 3750 2900 50  0000 L CNN
 F 1 "220 uf 25V" H 3750 2700 50  0000 L CNN
-F 2 "~" H 3700 2800 60  0000 C CNN
+F 2 "Capacitors_SMD:CP_Elec_8x10" H 3700 2800 60  0001 C CNN
 F 3 "~" H 3700 2800 60  0000 C CNN
 F 4 "647-UWT1E221MNL1GS" H 3700 2800 60  0001 C CNN "Mouser Part Number"
@@
 F 0 "L1" H 4550 3000 50  0000 C CNN
 F 1 "330 uh" H 4550 2850 50  0000 C CNN
-F 2 "~" H 4550 2900 60  0000 C CNN
+F 2 "SRN1060:SRN1060" H 4550 2900 60  0001 C CNN
 F 3 "~" H 4550 2900 60  0000 C CNN
 F 4 "652-SRN1060-331M" H 4550 2900 60  0001 C CNN "Mouser Part Number"
@@
 F 0 "D3" H 4850 3200 40  0000 C CNN
 F 1 "CMSH1-60 TR13" H 4850 3000 40  0000 C CNN
-F 2 "~" H 4850 3100 60  0000 C CNN
+F 2 "Diodes_SMD:D_SMB" H 4850 3100 60  0001 C CNN
 F 3 "~" H 4850 3100 60  0000 C CNN
 F 4 "610-CMSH1-60TR13" H 4850 3100 60  0001 C CNN "Mouser Part Number"
@@
 Connection ~ 4850 3300
 $Comp
-L GND #PWR015
+L GND-RESCUE-ESP32-PWMHalfSidingSMD #PWR015
 U 1 1 5C829DEF
 P 4850 3400
@@
 Wire Wire Line
 	4850 3300 4850 3400
-Text GLabel 5950 2550 0    100  Input ~ 0
+Text GLabel 5950 2550 2    50   Input ~ 0
 CAN +12V
 $EndSCHEMATC
