File: ESP32-PWMHalfSidingSMD/ESP32-PWMHalfSidingSMD.kicad_pcb (KiCad board)
At the start: 2 copper layers, 82.5 x 113 mm, 73 parts, among them IC1 MCT6H, IC2 MCT6H, J1 RJ45, J2 RJ45, P601 C A0 A1 A2 A3 A4 A5 A6 A7, P602 C B0 B1 B2 B3 B4 B5 B6 B7, Q1 MMBT3904, Q2 MMBT3904, T1 - 15 in +, T2 - 15 out +, T3 In Track1 Out, T4 Motor 1, T5 Motor 2, T6 In Track1 Out, T601 + 12V -, U0 ESP32_DEVKIT_C or TTGO-T1, U1 TCAN332DR, U3 LM2574N-5.0, U601 PCA9685, U602 TBD62X83A, U603 TBD62X83A, U7 TC4428, U8 TC4428, U9 74HCT00

Commit message: Updating 3D models in ESP32 PWM Half Siding.
Routing:
- net CAN +12V: track 173.9 -> 169.2 mm
- net Net-(D2-Pad2): track 4.93 -> 9.68 mm
Changed lines of the file:
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@@
   (general
     (links 218)
-    (no_connects 4)
-    (area 74.90163 20.160001 206.684286 157.64)
+    (no_connects 2)
+    (area 96.469999 30.429999 179.120001 143.560001)
     (thickness 1.6)
     (drawings 25)
@@
     (add_net Vdd)
   )
+  (module SOIC-8_N (layer F.Cu)
+    (at 137.16 60.96)
+    (descr "module CMS SOJ 8 pins etroit")
+    (tags "CMS SOJ")
+    (attr smd)
+    (fp_text reference U1 (at 0 -0.889) (layer F.SilkS)
+      (effects (font (size 1 1) (thickness 0.15)))
+    )
+    (fp_text value TCAN332DR (at 0 0.762) (layer F.SilkS)
+      (effects (font (size 0.8 0.8) (thickness 0.15)))
+    )
+    (fp_line (start -2.667 1.778) (end -2.667 1.905) (layer F.SilkS) (width 0.127))
+    (fp_line (start -2.667 1.905) (end 2.667 1.905) (layer F.SilkS) (width 0.127))
+    (fp_line (start 2.667 -1.905) (end -2.667 -1.905) (layer F.SilkS) (width 0.127))
+    (fp_line (start -2.667 -1.905) (end -2.667 1.778) (layer F.SilkS) (width 0.127))
+    (fp_line (start -2.667 -0.508) (end -2.159 -0.508) (layer F.SilkS) (width 0.127))
+    (fp_line (start -2.159 -0.508) (end -2.159 0.508) (layer F.SilkS) (width 0.127))
+    (fp_line (start -2.159 0.508) (end -2.667 0.508) (layer F.SilkS) (width 0.127))
+    (fp_line (start 2.667 -1.905) (end 2.667 1.905) (layer F.SilkS) (width 0.127))
+    (pad 8 smd rect (at -1.875 -2.7) (size 0.6 1.6) (layers F.Cu F.Paste F.Mask)
+      (net 116 "Net-(U1-Pad8)"))
+    (pad 1 smd rect (at -1.875 2.7) (size 0.6 1.6) (layers F.Cu F.Paste F.Mask)
+      (net 107 /CAN_TX))
+    (pad 7 smd rect (at -0.625 -2.7) (size 0.6 1.6) (layers F.Cu F.Paste F.Mask)
+      (net 3 "/CAN Transceiver/CANH"))
+    (pad 6 smd rect (at 0.625 -2.7) (size 0.6 1.6) (layers F.Cu F.Paste F.Mask)
+      (net 4 "/CAN Transceiver/CANL"))
+    (pad 5 smd rect (at 1.875 -2.7) (size 0.6 1.6) (layers F.Cu F.Paste F.Mask)
+      (net 117 "Net-(U1-Pad5)"))
+    (pad 2 smd rect (at -0.625 2.7) (size 0.6 1.6) (layers F.Cu F.Paste F.Mask)
+      (net 19 GND))
+    (pad 3 smd rect (at 0.625 2.7) (size 0.6 1.6) (layers F.Cu F.Paste F.Mask)
+      (net 17 3V3))
+    (pad 4 smd rect (at 1.875 2.7) (size 0.6 1.6) (layers F.Cu F.Paste F.Mask)
+      (net 105 /CAN_RX))
+    (model Housings_SOIC.3dshapes/SOIC-8_3.9x4.9mm_Pitch1.27mm.wrl
+      (at (xyz 0 0 0))
+      (scale (xyz 1 1 1))
+      (rotate (xyz 0 0 270))
+    )
+  )
   (module Diodes_SMD:D_SMB (layer F.Cu)
     (at 129.54 119.38 90)
@@
     )
   )
-  (module SOIC-8_N (layer F.Cu)
-    (at 137.16 60.96)
-    (descr "module CMS SOJ 8 pins etroit")
-    (tags "CMS SOJ")
-    (attr smd)
-    (fp_text reference U1 (at 0 -0.889) (layer F.SilkS)
-      (effects (font (size 1 1) (thickness 0.15)))
-    )
-    (fp_text value TCAN332DR (at 0 0.762) (layer F.SilkS)
-      (effects (font (size 0.8 0.8) (thickness 0.15)))
-    )
-    (fp_line (start -2.667 1.778) (end -2.667 1.905) (layer F.SilkS) (width 0.127))
-    (fp_line (start -2.667 1.905) (end 2.667 1.905) (layer F.SilkS) (width 0.127))
-    (fp_line (start 2.667 -1.905) (end -2.667 -1.905) (layer F.SilkS) (width 0.127))
-    (fp_line (start -2.667 -1.905) (end -2.667 1.778) (layer F.SilkS) (width 0.127))
-    (fp_line (start -2.667 -0.508) (end -2.159 -0.508) (layer F.SilkS) (width 0.127))
-    (fp_line (start -2.159 -0.508) (end -2.159 0.508) (layer F.SilkS) (width 0.127))
-    (fp_line (start -2.159 0.508) (end -2.667 0.508) (layer F.SilkS) (width 0.127))
-    (fp_line (start 2.667 -1.905) (end 2.667 1.905) (layer F.SilkS) (width 0.127))
-    (pad 8 smd rect (at -1.875 -2.7) (size 0.6 1.6) (layers F.Cu F.Paste F.Mask)
-      (net 116 "Net-(U1-Pad8)"))
-    (pad 1 smd rect (at -1.875 2.7) (size 0.6 1.6) (layers F.Cu F.Paste F.Mask)
-      (net 107 /CAN_TX))
-    (pad 7 smd rect (at -0.625 -2.7) (size 0.6 1.6) (layers F.Cu F.Paste F.Mask)
-      (net 3 "/CAN Transceiver/CANH"))
-    (pad 6 smd rect (at 0.625 -2.7) (size 0.6 1.6) (layers F.Cu F.Paste F.Mask)
-      (net 4 "/CAN Transceiver/CANL"))
-    (pad 5 smd rect (at 1.875 -2.7) (size 0.6 1.6) (layers F.Cu F.Paste F.Mask)
-      (net 117 "Net-(U1-Pad5)"))
-    (pad 2 smd rect (at -0.625 2.7) (size 0.6 1.6) (layers F.Cu F.Paste F.Mask)
-      (net 19 GND))
-    (pad 3 smd rect (at 0.625 2.7) (size 0.6 1.6) (layers F.Cu F.Paste F.Mask)
-      (net 17 3V3))
-    (pad 4 smd rect (at 1.875 2.7) (size 0.6 1.6) (layers F.Cu F.Paste F.Mask)
-      (net 105 /CAN_RX))
-    (model smd/cms_so8.wrl
-      (at (xyz 0 0 0))
-      (scale (xyz 0.5 0.32 0.5))
-      (rotate (xyz 0 0 0))
-    )
-  )
   (module tssop-28 (layer F.Cu)
     (at 163.83 96.52 180)
@@
   (segment (start 105.918 68.326) (end 105.918 65.786) (width 0.254) (layer F.Cu) (net 18))
   (segment (start 105.918 65.786) (end 105.664 65.532) (width 0.254) (layer F.Cu) (net 18))
-  (segment (start 160.118 41.91) (end 165.1 36.928) (width 0.508) (layer F.Cu) (net 18))
-  (segment (start 165.1 36.928) (end 165.1 35.79749) (width 0.508) (layer F.Cu) (net 18))
   (segment (start 149.479 45.72) (end 148.844 45.085) (width 0.508) (layer B.Cu) (net 18))
   (segment (start 146.44 41.91) (end 146.44 42.681) (width 0.508) (layer F.Cu) (net 18))
@@
   (segment (start 148.336 53.975) (end 148.59 54.229) (width 0.508) (layer B.Cu) (net 18))
   (segment (start 155.33 45.33) (end 154.94 45.72) (width 0.508) (layer F.Cu) (net 18))
+  (segment (start 155.33 41.91) (end 155.33 45.33) (width 0.508) (layer F.Cu) (net 18))
   (segment (start 146.05 127.5588) (end 146.05 123.444) (width 0.508) (layer F.Cu) (net 19))
   (via (at 145.796 123.19) (size 1.778) (drill 1.016) (layers F.Cu B.Cu) (net 19))
@@
   (segment (start 150.74 41.91) (end 150.74 39.76) (width 0.508) (layer F.Cu) (net 21))
   (segment (start 150.74 39.76) (end 156.21 34.29) (width 0.508) (layer F.Cu) (net 21))
-  (segment (start 155.33 41.91) (end 155.33 45.33) (width 0.508) (layer F.Cu) (net 22))
+  (segment (start 160.118 41.91) (end 165.1 36.928) (width 0.508) (layer F.Cu) (net 22))
+  (segment (start 165.1 36.928) (end 165.1 35.79749) (width 0.508) (layer F.Cu) (net 22))
   (segment (start 165.1 35.79749) (end 165.1 34.29) (width 0.508) (layer F.Cu) (net 22))
   (segment (start 129.54 121.53) (end 133.087 121.53) (width 0.508) (layer F.Cu) (net 23))
