File: ESP32-PWMHalfSidingSMD/PCA9685Driver.sch (KiCad schematic (older format))
At the start: 20 parts, among them P601 C A0 A1 A2 A3 A4 A5 A6 A7, P602 C B0 B1 B2 B3 B4 B5 B6 B7, T601 + 12V -, U601 PCA9685, U602 TBD62X83A, U603 TBD62X83A

Commit message: Generate BOM for ESP32-PWMHalfSidingSMD.
Parts:
- JP10, JP11, JP4, JP5, JP6, JP7, JP8, JP9: Mouser Part Number (none) -> 71-CRCW12060000Z0EBC
- JP2, JP3: Mouser Part Number (none) -> 71-CRCW06030000Z0EBC
- U601: Mouser Part Number 771-PCA9685PW,118 -> 771-PCA9685PW,118
- U602: Mouser Part Number 757-TBD62083AFG or 757-TBD62783AFG -> 757-TBD62083AFG or 757-TBD62783AFG
Changed lines of the file:
@@
 F 2 "" H 2800 2400 60  0001 C CNN
 F 3 "~" H 2800 2400 60  0000 C CNN
-F 4 " 771-PCA9685PW,118" H 2800 2400 60  0001 C CNN "Mouser Part Number"
+F 4 "771-PCA9685PW,118" H 2800 2400 60  0001 C CNN "Mouser Part Number"
 	1    2800 2400
 	1    0    0    -1
@@
 F 2 "" H 4800 1100 60  0001 C CNN
 F 3 "~" H 4800 1100 60  0000 C CNN
-F 4 " 757-TBD62083AFG or 757-TBD62783AFG" H 4800 1100 60  0001 C CNN "Mouser Part Number"
+F 4 "757-TBD62083AFG or 757-TBD62783AFG" H 4800 1100 60  0001 C CNN "Mouser Part Number"
 	1    4800 1100
 	1    0    0    -1
@@
 F 2 "Resistors_SMD:R_1206" V 4480 700 50  0001 C CNN
 F 3 "" H 4550 700 50  0001 C CNN
+F 4 "71-CRCW12060000Z0EBC" V 4550 700 60  0001 C CNN "Mouser Part Number"
 	1    4550 700
 	0    1    1    0
@@
 F 2 "Resistors_SMD:R_1206" V 4930 700 50  0001 C CNN
 F 3 "" H 5000 700 50  0001 C CNN
+F 4 "71-CRCW12060000Z0EBC" V 5000 700 60  0001 C CNN "Mouser Part Number"
 	1    5000 700
 	0    1    1    0
@@
 F 2 "Resistors_SMD:R_1206" V 4530 5150 50  0001 C CNN
 F 3 "" H 4600 5150 50  0001 C CNN
+F 4 "71-CRCW12060000Z0EBC" V 4600 5150 60  0001 C CNN "Mouser Part Number"
 	1    4600 5150
 	0    1    1    0
@@
 F 2 "Resistors_SMD:R_1206" V 4980 5150 50  0001 C CNN
 F 3 "" H 5050 5150 50  0001 C CNN
+F 4 "71-CRCW12060000Z0EBC" V 5050 5150 60  0001 C CNN "Mouser Part Number"
 	1    5050 5150
 	0    1    1    0
@@
 F 2 "Resistors_SMD:R_1206" V 7030 700 50  0001 C CNN
 F 3 "" H 7100 700 50  0001 C CNN
+F 4 "71-CRCW12060000Z0EBC" V 7100 700 60  0001 C CNN "Mouser Part Number"
 	1    7100 700
 	0    1    1    0
@@
 F 2 "Resistors_SMD:R_1206" V 7430 700 50  0001 C CNN
 F 3 "" H 7500 700 50  0001 C CNN
+F 4 "71-CRCW12060000Z0EBC" V 7500 700 60  0001 C CNN "Mouser Part Number"
 	1    7500 700
 	0    1    1    0
@@
 F 2 "Resistors_SMD:R_1206" V 7030 5100 50  0001 C CNN
 F 3 "" H 7100 5100 50  0001 C CNN
+F 4 "71-CRCW12060000Z0EBC" V 7100 5100 60  0001 C CNN "Mouser Part Number"
 	1    7100 5100
 	0    1    1    0
@@
 F 2 "Resistors_SMD:R_1206" V 7480 5100 50  0001 C CNN
 F 3 "" H 7550 5100 50  0001 C CNN
+F 4 "71-CRCW12060000Z0EBC" V 7550 5100 60  0001 C CNN "Mouser Part Number"
 	1    7550 5100
 	0    1    1    0
@@
 F 2 "Resistors_SMD:R_0603" V 2480 3050 50  0001 C CNN
 F 3 "" H 2550 3050 50  0001 C CNN
+F 4 "71-CRCW06030000Z0EBC" V 2550 3050 60  0001 C CNN "Mouser Part Number"
 	1    2550 3050
 	0    1    1    0
@@
 F 2 "Resistors_SMD:R_0603" V 1430 3350 50  0001 C CNN
 F 3 "" H 1500 3350 50  0001 C CNN
+F 4 "71-CRCW06030000Z0EBC" V 1500 3350 60  0001 C CNN "Mouser Part Number"
 	1    1500 3350
 	0    1    1    0

Commit message: Update footprints in ESP32-PWMHalfSidingSMD.
Parts:
- U601: footprint (none) -> Housings_SSOP:TSSOP-28_4.4x9.7mm_Pitch0.65mm
- U602, U603: footprint (none) -> Housings_SOIC:SOIC-18W_7.5x11.6mm_Pitch1.27mm
Changed lines of the file:
@@
 F 0 "U601" H 2800 2200 60  0000 C CNN
 F 1 "PCA9685" V 2800 2500 60  0000 C CNN
-F 2 "" H 2800 2400 60  0001 C CNN
+F 2 "Housings_SSOP:TSSOP-28_4.4x9.7mm_Pitch0.65mm" H 2800 2400 60  0001 C CNN
 F 3 "~" H 2800 2400 60  0000 C CNN
 F 4 "771-PCA9685PW,118" H 2800 2400 60  0001 C CNN "Mouser Part Number"
@@
 F 0 "U602" H 4900 950 60  0000 C CNN
 F 1 "TBD62X83A" H 5050 1200 60  0000 C CNN
-F 2 "" H 4800 1100 60  0001 C CNN
+F 2 "Housings_SOIC:SOIC-18W_7.5x11.6mm_Pitch1.27mm" H 4800 1100 60  0001 C CNN
 F 3 "~" H 4800 1100 60  0000 C CNN
 F 4 "757-TBD62083AFG or 757-TBD62783AFG" H 4800 1100 60  0001 C CNN "Mouser Part Number"
@@
 F 0 "U603" H 7400 900 60  0000 C CNN
 F 1 "TBD62X83A" H 7550 1150 60  0000 C CNN
-F 2 "" H 7300 1050 60  0001 C CNN
+F 2 "Housings_SOIC:SOIC-18W_7.5x11.6mm_Pitch1.27mm" H 7300 1050 60  0001 C CNN
 F 3 "~" H 7300 1050 60  0000 C CNN
 F 4 "757-TBD62083AFG or 757-TBD62783AFG" H 7300 1050 60  0001 C CNN "Mouser Part Number"
