File: ESP32-PWMHalfSidingSMD/OD1.sch (KiCad schematic (older format))
At the start: 5 parts, among them IC1 MCT6H, T3 In Track1 Out

Commit message: Update part numbers for ESP32-PWMHalfSidingSMD and created prelim BOM files.
Parts:
- R3: Mouser Part Number 603-CFR-25JR-5210R -> 71-CRCW060310R0FKEAC
- R4: Mouser Part Number 603-CFR25SJT-52-10K -> 71-CRCW060310K0JNEBC
Changed lines of the file:
@@
 F 2 "~" V 2430 1500 30  0000 C CNN
 F 3 "~" H 2500 1500 30  0000 C CNN
-F 4 "603-CFR-25JR-5210R" H 2500 1500 60  0001 C CNN "Mouser Part Number"
+F 4 "71-CRCW060310R0FKEAC" H 2500 1500 60  0001 C CNN "Mouser Part Number"
 	1    2500 1500
 	0    -1   -1   0
@@
 F 2 "~" V 4230 1100 30  0000 C CNN
 F 3 "~" H 4300 1100 30  0000 C CNN
-F 4 "603-CFR25SJT-52-10K" H 4300 1100 60  0001 C CNN "Mouser Part Number"
+F 4 "71-CRCW060310K0JNEBC" H 4300 1100 60  0001 C CNN "Mouser Part Number"
 	1    4300 1100
 	1    0    0    -1

Commit message: Repair ESP32-PWMHalfSidingSMD and generate POS file.
Parts:
- added D6: LED, LEDs:LED_0603, symbol LED
- added Q1: MMBT3904, TO_SOT_Packages_SMD:SOT-23, symbol MMBT3904
- D4: footprint ~ -> Z4DGP:Z4DGP
- IC1: footprint DIP-8__300 -> SMT8:SMT8
- R3: footprint ~ -> Resistors_SMD:R_0603; symbol R -> R-RESCUE-ESP32-PWMHalfSidingSMD
- R4: value 10K Ohms -> 2.7K Ohms; footprint ~ -> Resistors_SMD:R_0603; symbol R -> R-RESCUE-ESP32-PWMHalfSidingSMD
- T3: footprint ~ -> Connectors:bornier2
Connections:
- wire segments 22 -> 28
Other:
- moved on the sheet: R4
Changed lines of the file:
@@
 EESchema Schematic File Version 2
+LIBS:ESP32-PWMHalfSidingSMD-rescue
 LIBS:power
 LIBS:device
@@
 LIBS:memory
 LIBS:xilinx
-LIBS:special
 LIBS:microcontrollers
 LIBS:dsp
@@
 LIBS:4814p-2
 LIBS:ESP32-PWMHalfSidingSMD-cache
-EELAYER 27 0
+EELAYER 25 0
 EELAYER END
 $Descr A4 11693 8268
@@
 F 0 "T3" V 1300 1300 40  0000 C CNN
 F 1 "In Track1 Out" V 1400 1300 40  0000 C CNN
-F 2 "~" H 1350 1300 60  0000 C CNN
+F 2 "Connectors:bornier2" H 1350 1300 60  0001 C CNN
 F 3 "~" H 1350 1300 60  0000 C CNN
 F 4 " 490-TB007-508-02BE" H 1350 1300 60  0001 C CNN "Mouser Part Number"
@@
 $EndComp
 $Comp
-L R R?
+L R-RESCUE-ESP32-PWMHalfSidingSMD R?
 U 1 1 5C831701
 P 2500 1500
@@
 F 0 "R3" V 2580 1500 40  0000 C CNN
 F 1 "10 Ohms" V 2507 1501 40  0000 C CNN
-F 2 "~" V 2430 1500 30  0000 C CNN
+F 2 "Resistors_SMD:R_0603" V 2430 1500 30  0001 C CNN
 F 3 "~" H 2500 1500 30  0000 C CNN
 F 4 "71-CRCW060310R0FKEAC" H 2500 1500 60  0001 C CNN "Mouser Part Number"
@@
 F 0 "IC1" H 3490 1790 40  0000 C CNN
 F 1 "MCT6H" H 3810 1410 40  0000 C CNN
-F 2 "DIP-8__300" H 3540 1420 30  0001 C CIN
+F 2 "SMT8:SMT8" H 3540 1420 30  0001 C CIN
 F 3 "~" H 3700 1600 60  0000 C CNN
 F 4 " MCT6SD" H 3700 1600 60  0001 C CNN "Mouser Part Number"
@@
 F 0 "IC1" H 3490 2340 40  0000 C CNN
 F 1 "MCT6H" H 3810 1960 40  0000 C CNN
-F 2 "DIP-8__300" H 3540 1970 30  0001 C CIN
+F 2 "SMT8:SMT8" H 3540 1970 30  0001 C CIN
 F 3 "~" H 3700 2150 60  0000 C CNN
 F 4 "MCT6SD" H 3700 2150 60  0001 C CNN "Mouser Part Number"
@@
 $EndComp
 $Comp
-L R R?
+L R-RESCUE-ESP32-PWMHalfSidingSMD R?
 U 1 1 5C831709
-P 4300 1100
+P 4950 900
 AR Path="/5C70A8FB/5C831709" Ref="R?"  Part="1"
 AR Path="/5C70AEE5/5C831709" Ref="R?"  Part="1"
 AR Path="/5C7DB984/5C831709" Ref="R?"  Part="1"
 AR Path="/5CA26382/5C831709" Ref="R4"  Part="1"
-F 0 "R4" V 4380 1100 40  0000 C CNN
-F 1 "10K Ohms" V 4307 1101 40  0000 C CNN
-F 2 "~" V 4230 1100 30  0000 C CNN
-F 3 "~" H 4300 1100 30  0000 C CNN
-F 4 "71-CRCW060310K0JNEBC" H 4300 1100 60  0001 C CNN "Mouser Part Number"
-	1    4300 1100
+F 0 "R4" V 5030 900 40  0000 C CNN
+F 1 "2.7K Ohms" V 4957 901 40  0000 C CNN
+F 2 "Resistors_SMD:R_0603" V 4880 900 30  0001 C CNN
+F 3 "~" H 4950 900 30  0000 C CNN
+F 4 "71-CRCW060310K0JNEBC" H 4950 900 60  0001 C CNN "Mouser Part Number"
+	1    4950 900
 	1    0    0    -1
 $EndComp
@@
 F 0 "D4" H 2050 3000 70  0000 C CNN
 F 1 "BRIDGEX" H 2050 2900 70  0000 C CNN
-F 2 "~" H 2050 2950 60  0000 C CNN
+F 2 "Z4DGP:Z4DGP" H 2050 2950 60  0001 C CNN
 F 3 "~" H 2050 2950 60  0000 C CNN
 F 4 "Z4DGP406L-HF" H 2050 2950 60  0001 C CNN "Mouser Part Number"
@@
 	4300 2050 4050 2050
 Wire Wire Line
-	4300 1350 4300 2050
-Wire Wire Line
-	4050 1500 4450 1500
+	4300 750  4300 2050
 Wire Wire Line
 	4050 1700 4200 1700
 Wire Wire Line
-	4200 1700 4200 2450
-Wire Wire Line
-	4200 2250 4050 2250
+	4050 2250 4650 2250
 Connection ~ 3200 1500
 Wire Wire Line
 	3350 1850 2900 1850
 Connection ~ 3350 1850
-Connection ~ 4300 1500
 $Comp
 L 3V3 #PWR015
@@
 	1    0    0    -1
 $EndComp
-Wire Wire Line
-	4300 750  4300 850
-$Comp
-L GND #PWR016
+$Comp
+L GND-RESCUE-ESP32-PWMHalfSidingSMD #PWR016
 U 1 1 5C831711
-P 4200 2450
+P 4950 2600
 AR Path="/5C70A8FB/5C831711" Ref="#PWR016"  Part="1"
 AR Path="/5C70AEE5/5C831711" Ref="#PWR?"  Part="1"
 AR Path="/5C7DB984/5C831711" Ref="#PWR015"  Part="1"
 AR Path="/5CA26382/5C831711" Ref="#PWR018"  Part="1"
-F 0 "#PWR018" H 4200 2450 30  0001 C CNN
-F 1 "GND" H 4200 2380 30  0001 C CNN
-F 2 "" H 4200 2450 60  0000 C CNN
-F 3 "" H 4200 2450 60  0000 C CNN
-	1    4200 2450
-	1    0    0    -1
-$EndComp
-Connection ~ 4200 2250
-Text HLabel 4450 1500 2    60   Input ~ 0
+F 0 "#PWR018" H 4950 2600 30  0001 C CNN
+F 1 "GND" H 4950 2530 30  0001 C CNN
+F 2 "" H 4950 2600 60  0000 C CNN
+F 3 "" H 4950 2600 60  0000 C CNN
+	1    4950 2600
+	1    0    0    -1
+$EndComp
+Text HLabel 5800 1900 2    60   Input ~ 0
 OD1
 Wire Wire Line
@@
 Wire Wire Line
 	1200 2450 1200 2950
+$Comp
+L MMBT3904 Q1
+U 1 1 608BDCD4
+P 4850 2250
+F 0 "Q1" H 5050 2325 50  0000 L CNN
+F 1 "MMBT3904" H 5050 2250 50  0000 L CNN
+F 2 "TO_SOT_Packages_SMD:SOT-23" H 5050 2175 50  0001 L CIN
+F 3 "" H 4850 2250 50  0001 L CNN
+	1    4850 2250
+	1    0    0    -1
+$EndComp
+$Comp
+L LED D6
+U 1 1 608BDE22
+P 4950 1600
+F 0 "D6" H 4950 1700 50  0000 C CNN
+F 1 "LED" H 4950 1500 50  0000 C CNN
+F 2 "LEDs:LED_0603" H 4950 1600 50  0001 C CNN
+F 3 "" H 4950 1600 50  0001 C CNN
+	1    4950 1600
+	0    -1   -1   0
+$EndComp
+Wire Wire Line
+	4050 1500 4300 1500
+Connection ~ 4300 1500
+Wire Wire Line
+	4200 1700 4200 2250
+Connection ~ 4200 2250
+Wire Wire Line
+	4950 2450 4950 2600
+Wire Wire Line
+	4950 1150 4950 1450
+Wire Wire Line
+	4950 1750 4950 2050
+Wire Wire Line
+	5800 1900 4950 1900
+Connection ~ 4950 1900
+Wire Wire Line
+	4950 650  4700 650
+Wire Wire Line
+	4700 650  4700 850
+Wire Wire Line
+	4700 850  4300 850
+Connection ~ 4300 850
 $EndSCHEMATC

Commit message: Generate BOM for ESP32-PWMHalfSidingSMD.
Parts:
- D4: Mouser Part Number Z4DGP406L-HF -> 750-Z4DGP406L-HF
- D6: Mouser Part Number (none) -> 710-150060SS55040
- IC1: Mouser Part Number MCT6SD -> 512-MCT6SD
- Q1: Mouser Part Number (none) -> 771-MMBT3904T/R
- R4: Mouser Part Number 71-CRCW060310K0JNEBC -> 71-CRCW06032K70JNEAC
- T3: Mouser Part Number 490-TB007-508-02BE -> 490-TB007-508-02BE
Changed lines of the file:
@@
 F 2 "Connectors:bornier2" H 1350 1300 60  0001 C CNN
 F 3 "~" H 1350 1300 60  0000 C CNN
-F 4 " 490-TB007-508-02BE" H 1350 1300 60  0001 C CNN "Mouser Part Number"
+F 4 "490-TB007-508-02BE" H 1350 1300 60  0001 C CNN "Mouser Part Number"
 	1    1350 1300
 	0    -1   -1   0
@@
 F 2 "SMT8:SMT8" H 3540 1420 30  0001 C CIN
 F 3 "~" H 3700 1600 60  0000 C CNN
-F 4 " MCT6SD" H 3700 1600 60  0001 C CNN "Mouser Part Number"
+F 4 "512-MCT6SD" H 3700 1600 60  0001 C CNN "Mouser Part Number"
 	1    3700 1600
 	1    0    0    -1
@@
 F 2 "Resistors_SMD:R_0603" V 4880 900 30  0001 C CNN
 F 3 "~" H 4950 900 30  0000 C CNN
-F 4 "71-CRCW060310K0JNEBC" H 4950 900 60  0001 C CNN "Mouser Part Number"
+F 4 "71-CRCW06032K70JNEAC" H 4950 900 60  0001 C CNN "Mouser Part Number"
 	1    4950 900
 	1    0    0    -1
@@
 F 2 "Z4DGP:Z4DGP" H 2050 2950 60  0001 C CNN
 F 3 "~" H 2050 2950 60  0000 C CNN
-F 4 "Z4DGP406L-HF" H 2050 2950 60  0001 C CNN "Mouser Part Number"
+F 4 "750-Z4DGP406L-HF " H 2050 2950 60  0001 C CNN "Mouser Part Number"
 	1    2050 2950
 	0    1    1    0
@@
 F 2 "TO_SOT_Packages_SMD:SOT-23" H 5050 2175 50  0001 L CIN
 F 3 "" H 4850 2250 50  0001 L CNN
+F 4 "771-MMBT3904T/R" H 4850 2250 60  0001 C CNN "Mouser Part Number"
 	1    4850 2250
 	1    0    0    -1
@@
 F 2 "LEDs:LED_0603" H 4950 1600 50  0001 C CNN
 F 3 "" H 4950 1600 50  0001 C CNN
+F 4 "710-150060SS55040" H 4950 1600 60  0001 C CNN "Mouser Part Number"
 	1    4950 1600
 	0    -1   -1   0

Commit message: Updates to ESP32-PWMHalfSidingSMD: I2C pullups, alt. SCL pins.
Changed lines of the file:
@@
 AR Path="/5C70AEE5/5C83170E" Ref="#PWR?"  Part="1"
 AR Path="/5C7DB984/5C83170E" Ref="#PWR014"  Part="1"
-AR Path="/5CA26382/5C83170E" Ref="#PWR017"  Part="1"
-F 0 "#PWR017" H 4300 710 30  0001 C CNN
+AR Path="/5CA26382/5C83170E" Ref="#PWR018"  Part="1"
+F 0 "#PWR018" H 4300 710 30  0001 C CNN
 F 1 "3V3" H 4300 860 30  0000 C CNN
 F 2 "" H 4300 750 60  0000 C CNN
@@
 AR Path="/5C70AEE5/5C831711" Ref="#PWR?"  Part="1"
 AR Path="/5C7DB984/5C831711" Ref="#PWR015"  Part="1"
-AR Path="/5CA26382/5C831711" Ref="#PWR018"  Part="1"
-F 0 "#PWR018" H 4950 2600 30  0001 C CNN
+AR Path="/5CA26382/5C831711" Ref="#PWR019"  Part="1"
+F 0 "#PWR019" H 4950 2600 30  0001 C CNN
 F 1 "GND" H 4950 2530 30  0001 C CNN
 F 2 "" H 4950 2600 60  0000 C CNN
@@
 	4950 1150 4950 1450
 Wire Wire Line
-	4950 1750 4950 2050
-Wire Wire Line
-	5800 1900 4950 1900
-Connection ~ 4950 1900
-Wire Wire Line
 	4950 650  4700 650
 Wire Wire Line
@@
 	4700 850  4300 850
 Connection ~ 4300 850
+Wire Wire Line
+	4950 2050 4950 1750
+Wire Wire Line
+	5800 1900 4950 1900
+Connection ~ 4950 1900
 $EndSCHEMATC
