File: ESP32-D0WD-V3-MultiFunction/Buttons4LEDs4.sch (KiCad schematic (older format))
At the start: 22 parts, among them U401 TC4426, U402 TC4426, U403 74HCT14

Commit message: Complete BOM for ESP32-D0WD-V3-MultiFunction.
Parts:
- U401, U402: Mouser Part Number (none) -> 579-TC1426COA713
Changed lines of the file:
@@
 encoding utf-8
 Sheet 4 8
-Title "ESP32 Multifunction board"
+Title "ESP32 Multifunction Board"
 Date ""
-Rev ""
+Rev "1.0"
 Comp "Deepwoods Software"
 Comment1 "Generic Buttons and LEDs"
@@
 F 2 "Housings_SOIC:SOIC-8_3.9x4.9mm_Pitch1.27mm" H 2500 3400 60  0001 C CNN
 F 3 "" H 2500 3400 60  0000 C CNN
+F 4 "579-TC1426COA713" H 2500 3400 60  0001 C CNN "Mouser Part Number"
 	1    2500 3400
 	1    0    0    -1
@@
 F 2 "Housings_SOIC:SOIC-8_3.9x4.9mm_Pitch1.27mm" H 2500 4250 60  0001 C CNN
 F 3 "" H 2500 4250 60  0000 C CNN
+F 4 "579-TC1426COA713" H 2500 4250 60  0001 C CNN "Mouser Part Number"
 	2    2500 4250
 	1    0    0    -1
@@
 F 2 "Housings_SOIC:SOIC-8_3.9x4.9mm_Pitch1.27mm" H 2450 1800 60  0001 C CNN
 F 3 "" H 2450 1800 60  0000 C CNN
+F 4 "579-TC1426COA713" H 2450 1800 60  0001 C CNN "Mouser Part Number"
 	1    2450 1800
 	1    0    0    -1
@@
 F 2 "Housings_SOIC:SOIC-8_3.9x4.9mm_Pitch1.27mm" H 2450 2600 60  0001 C CNN
 F 3 "" H 2450 2600 60  0000 C CNN
+F 4 "579-TC1426COA713" H 2450 2600 60  0001 C CNN "Mouser Part Number"
 	2    2450 2600
 	1    0    0    -1
