File: ESP32-D0WD-V3-MultiFunction/OccDetect4.sch (KiCad schematic (older format))
At the start: 35 parts, among them U601 LM339, U602 LM339

Commit message: Complete BOM for ESP32-D0WD-V3-MultiFunction.
Parts:
- U601, U602: Mouser Part Number (none) -> 595-LM339DR
Changed lines of the file:
@@
 encoding utf-8
 Sheet 6 8
-Title "ESP32 Multifunction board"
+Title "ESP32 Multifunction Board"
 Date ""
-Rev ""
+Rev "1.0"
 Comp "Deepwoods Software"
 Comment1 "Occupancy Detectors"
@@
 F 2 "Housings_SOIC:SOIC-14_3.9x8.7mm_Pitch1.27mm" H 3250 1700 50  0001 C CNN
 F 3 "" H 3350 1800 50  0001 C CNN
+F 4 "595-LM339DR" H 3300 1600 60  0001 C CNN "Mouser Part Number"
 	1    3300 1600
 	1    0    0    -1
@@
 F 2 "Housings_SOIC:SOIC-14_3.9x8.7mm_Pitch1.27mm" H 4400 1800 50  0001 C CNN
 F 3 "" H 4500 1900 50  0001 C CNN
+F 4 "595-LM339DR" H 4450 1700 60  0001 C CNN "Mouser Part Number"
 	1    4450 1700
 	1    0    0    -1
