File: ESP32-D0WD-V3-MultiFunction/PCA9685Driver.sch (KiCad schematic (older format))
At the start: 18 parts, among them P701 A7 A6 A5 A4 A3 A2 A1 A0 C, P702 B7 B6 B5 B4 B3 B2 B1 B0 C, T701 + 12V -, U701 PCA9685, U702 TBD62X83A, U703 TBD62X83A

Commit message: Fixed footprints for DFLS240-7s.
Parts:
- D701: footprint Diodes_SMD:D_SMB -> Diodes_SMD:D_PowerDI-123
Changed lines of the file:
@@
 F 0 "D701" H 3500 5150 40  0000 C CNN
 F 1 "DFLS240-7" H 3500 4950 40  0000 C CNN
-F 2 "Diodes_SMD:D_SMB" H 3500 5050 60  0001 C CNN
+F 2 "Diodes_SMD:D_PowerDI-123" H 3500 5050 60  0001 C CNN
 F 3 "~" H 3500 5050 60  0000 C CNN
 F 4 "621-DFLS240-7" H 3500 5050 60  0001 C CNN "Mouser Part Number"
