File: ESP32-D0WD-V3-USBProgBoard/ESP32-D0WD-V3-USBProgBoard.kicad_pcb (KiCad board)
At the start: 2 copper layers, 21.6 x 41.9 mm, 27 parts, among them J1 USB_OTG, J2 ProgHeader, Q1 SSM3J117TU, Q2 UMH3N, U1 FT231XS-R, U2 TC1263-3.3VOATR

Commit message: Final touches on USB prog board.
Parts:
- added ?: , DWSLogoBCU:DWSLogoBCU, F.Cu at (98.9, 91.8)
- added REF**: Fiducial_classic_Small_SilkscreenTop_Type1, Fiducials:Fiducial_classic_Small_SilkscreenTop_Type1, F.Cu at (99.3, 98.2)
- added REF**: Fiducial_classic_Small_SilkscreenTop_Type1, Fiducials:Fiducial_classic_Small_SilkscreenTop_Type1, F.Cu at (93.0, 72.9)
- added REF**: Fiducial_classic_Small_SilkscreenTop_Type1, Fiducials:Fiducial_classic_Small_SilkscreenTop_Type1, F.Cu at (84.8, 67.6)
- added REF***: OSHW-Logo2_7.3x6mm_SilkScreen, Symbols:OSHW-Logo2_7.3x6mm_SilkScreen, F.Cu at (99.1, 90.3)
