File: LCCCANCape/LCCCANCape.kicad_pcb (KiCad board)
At the start: 2 copper layers, 54.6 x 98.3 mm, 27 parts, among them J1 RJ45, J2 RJ45, J3 Console Feed Through, P8 BeagleBone_Black_Header, P9 BeagleBone_Black_Header, T1 + 15 in -, T2 + 15 out -, U2 CAT24C256W, U3 TCAN332DR

Commit message: Finalize for PCBWay.
Parts:
- moved R3 3.18 mm to (136.0, 114.9)
- moved R2 3.05 mm to (136.0, 123.7)
- moved JP1 0.38 mm to (124.0, 75.1)
Routing:
- net Net-(JMP1-Pad2): track 2.18 -> 5.38 mm
- net Net-(JMP1-Pad1): track 2.18 -> 5.25 mm
Other:
- net class Default removed

Commit message: Finalize for PCBWay.
Parts:
- added G***: LOGO, DWS:DWSLogoBCU, F.Cu at (154.9, 76.2)
- added G***: LCC, LCC:LCC_LOGO_4.5x4.5, F.Cu at (125.7, 118.1)
- added REF**: KiCad-Logo2_5mm_SilkScreen, Symbol:KiCad-Logo2_5mm_SilkScreen, F.Cu at (129.5, 67.3)
- added REF**: WEEE-Logo_5.6x8mm_SilkScreen, Symbol:WEEE-Logo_5.6x8mm_SilkScreen, F.Cu at (157.5, 57.1)
- added REF**: OSHW-Logo2_7.3x6mm_SilkScreen, Symbol:OSHW-Logo2_7.3x6mm_SilkScreen, F.Cu at (142.2, 68.6)
- added REF**: PowerLabel-00, PowerLab:PowerLabel-00, F.Cu at (156.2, 118.1)
- added REF**: ESD-Logo_13.2x12mm_SilkScreen, Symbol:ESD-Logo_13.2x12mm_SilkScreen, F.Cu at (127.0, 52.1)
Other:
- board text added: "(C) 2023 Robert Heller D/B/A Deepwoods Software LCC CAN CAPE (SMD) Rev. B"

Commit message: Add 3D shapes to SMD version.
Parts:
- T1, T2: footprint Connectors_Terminal_Blocks:TerminalBlock_Pheonix_MPT-2.54mm_2pol -> Connectors_Terminal_Blocks:TerminalBlock_Phoenix_MPT-2.54mm_2pol
Changed lines of the file:
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@@
     (pad "46" thru_hole oval locked (at 2.54 55.88) (size 1.7272 1.7272) (drill 1.016) (layers *.Cu *.Mask "F.SilkS")
       (net 69 "Net-(P8-Pad46)"))
-    (model "Pin_Headers.3dshapes/Pin_Header_Straight_2x23_Pitch2.54mm.wrl"
+    (model "${KICAD6_3DMODEL_DIR}/Connector_PinHeader_2.54mm.3dshapes/PinHeader_2x23_P2.54mm_Vertical.wrl"
       (offset (xyz 0 -55.87999916 -1.269999981))
       (scale (xyz 1 1 1))
@@
     (pad "46" thru_hole oval locked (at 2.54 55.88) (size 1.7272 1.7272) (drill 1.016) (layers *.Cu *.Mask "F.SilkS")
       (net 7 "GND"))
-    (model "Pin_Headers.3dshapes/Pin_Header_Straight_2x23_Pitch2.54mm.wrl"
+    (model "${KICAD6_3DMODEL_DIR}/Connector_PinHeader_2.54mm.3dshapes/PinHeader_2x23_P2.54mm_Vertical.wrl"
       (offset (xyz 0 -55.87999916 -1.269999981))
       (scale (xyz 1 1 1))
@@
     (pad "8" thru_hole circle locked (at 4.445 -8.89 270) (size 1.50114 1.50114) (drill 0.89916) (layers *.Cu *.Mask "F.SilkS")
       (net 11 "Net-(D2-Pad2)"))
-    (model "Connectors.3dshapes/RJ45_8.wrl"
-      (offset (xyz 0 0 0))
-      (scale (xyz 0.4 0.4 0.4))
-      (rotate (xyz 0 0 0))
+    (model "${KIPRJMOD}/WURTH_615008144221.wrl"
+      (offset (xyz 0 1.5 7.5))
+      (scale (xyz 390 390 390))
+      (rotate (xyz -90 0 0))
     )
   )
@@
     (pad "8" thru_hole circle locked (at 4.445 -8.89 90) (size 1.50114 1.50114) (drill 0.89916) (layers *.Cu *.Mask "F.SilkS")
       (net 11 "Net-(D2-Pad2)"))
-    (model "Connectors.3dshapes/RJ45_8.wrl"
-      (offset (xyz 0 0 0))
-      (scale (xyz 0.4 0.4 0.4))
-      (rotate (xyz 0 0 0))
+    (model "${KIPRJMOD}/WURTH_615008144221.wrl"
+      (offset (xyz 0 1.5 7.5))
+      (scale (xyz 390 390 390))
+      (rotate (xyz -90 0 0))
     )
   )
@@
     (pad "4" thru_hole oval locked (at 2.54 2.54 90) (size 1.7 1.7) (drill 1) (layers *.Cu *.Mask)
       (net 9 "Net-(C3-Pad1)"))
-    (model "${KISYS3DMOD}/Pin_Headers.3dshapes/Pin_Header_Straight_2x02_Pitch2.54mm.wrl"
+    (model "${KICAD6_3DMODEL_DIR}/Connector_PinHeader_2.54mm.3dshapes/PinHeader_2x02_P2.54mm_Vertical.wrl"
       (offset (xyz 0 0 0))
       (scale (xyz 1 1 1))
@@
     (pad "8" smd rect locked (at 2.7 -1.905 180) (size 1.55 0.6) (layers "F.Cu" "F.Paste" "F.Mask")
       (net 103 "Net-(U3-Pad8)"))
-    (model "${KISYS3DMOD}/Housings_SOIC.3dshapes/SOIC-8_3.9x4.9mm_Pitch1.27mm.wrl"
+    (model "${KICAD6_3DMODEL_DIR}/Package_SO.3dshapes/SOIC-8_3.9x4.9mm_P1.27mm.wrl"
       (offset (xyz 0 0 0))
       (scale (xyz 1 1 1))
@@
     (pad "2" smd rect locked (at 0.75 0 270) (size 0.8 0.75) (layers "F.Cu" "F.Paste" "F.Mask")
       (net 7 "GND"))
-    (model "Capacitors_SMD.3dshapes/C_0603.wrl"
+    (model "${KICAD6_3DMODEL_DIR}/Capacitor_SMD.3dshapes/C_0603_1608Metric.wrl"
       (offset (xyz 0 0 0))
       (scale (xyz 1 1 1))
@@
     (pad "2" smd rect locked (at 1.8 0 90) (size 2.6 1.6) (layers "F.Cu" "F.Paste" "F.Mask")
       (net 7 "GND"))
-    (model "Capacitors_SMD.3dshapes/CP_Elec_4x5.7.wrl"
+    (model "${KICAD6_3DMODEL_DIR}/Capacitor_SMD.3dshapes/CP_Elec_4x5.7.wrl"
       (offset (xyz 0 0 0))
       (scale (xyz 1 1 1))
@@
     (pad "2" smd rect locked (at 0.75 0) (size 0.8 0.75) (layers "F.Cu" "F.Paste" "F.Mask")
       (net 7 "GND"))
-    (model "Capacitors_SMD.3dshapes/C_0603.wrl"
+    (model "${KICAD6_3DMODEL_DIR}/Capacitor_SMD.3dshapes/C_0603_1608Metric.wrl"
       (offset (xyz 0 0 0))
       (scale (xyz 1 1 1))
@@
     (pad "2" smd rect locked (at 0.75 0 180) (size 0.8 0.75) (layers "F.Cu" "F.Paste" "F.Mask")
       (net 7 "GND"))
-    (model "Capacitors_SMD.3dshapes/C_0603.wrl"
+    (model "${KICAD6_3DMODEL_DIR}/Capacitor_SMD.3dshapes/C_0603_1608Metric.wrl"
       (offset (xyz 0 0 0))
       (scale (xyz 1 1 1))
@@
     (pad "2" smd rect locked (at 1.525 0) (size 1.05 1.5) (layers "F.Cu" "F.Paste" "F.Mask")
       (net 11 "Net-(D2-Pad2)"))
-    (model "${KISYS3DMOD}/Diodes_SMD.3dshapes/D_PowerDI-123.wrl"
+    (model "${KICAD6_3DMODEL_DIR}/Diode_SMD.3dshapes/D_PowerDI-123.wrl"
       (offset (xyz 0 0 0))
       (scale (xyz 1 1 1))
@@
     (pad "2" smd rect locked (at 1.525 0 180) (size 1.05 1.5) (layers "F.Cu" "F.Paste" "F.Mask")
       (net 12 "Net-(D3-Pad2)"))
-    (model "${KISYS3DMOD}/Diodes_SMD.3dshapes/D_PowerDI-123.wrl"
+    (model "${KICAD6_3DMODEL_DIR}/Diode_SMD.3dshapes/D_PowerDI-123.wrl"
       (offset (xyz 0 0 0))
       (scale (xyz 1 1 1))
@@
     (pad "6" thru_hole oval locked (at 0 12.7) (size 1.7 1.7) (drill 1) (layers *.Cu *.Mask)
       (net 20 "Net-(J3-Pad6)"))
-    (model "${KISYS3DMOD}/Pin_Headers.3dshapes/Pin_Header_Straight_1x06_Pitch2.54mm.wrl"
+    (model "${KICAD6_3DMODEL_DIR}/Pin_Headers.3dshapes/Pin_Header_Straight_1x06_Pitch2.54mm.wrl"
       (offset (xyz 0 0 -3.809999943))
       (scale (xyz 1 1 1))
@@
     (pad "2" smd rect locked (at 1.45 0) (size 0.9 1.7) (layers "F.Cu" "F.Paste" "F.Mask")
       (net 21 "Net-(JMP1-Pad1)"))
-    (model "${KISYS3DMOD}/Resistors_SMD.3dshapes/R_1206.wrl"
+    (model "${KICAD6_3DMODEL_DIR}/Resistor_SMD.3dshapes/R_1206_3216Metric.wrl"
       (offset (xyz 0 0 0))
       (scale (xyz 1 1 1))
@@
     (pad "2" smd rect locked (at 1.45 0) (size 0.9 1.7) (layers "F.Cu" "F.Paste" "F.Mask")
       (net 22 "Net-(JMP1-Pad2)"))
-    (model "${KISYS3DMOD}/Resistors_SMD.3dshapes/R_1206.wrl"
+    (model "${KICAD6_3DMODEL_DIR}/Resistor_SMD.3dshapes/R_1206_3216Metric.wrl"
       (offset (xyz 0 0 0))
       (scale (xyz 1 1 1))
@@
     (pad "2" smd rect locked (at 0.75 0 90) (size 0.5 0.9) (layers "F.Cu" "F.Paste" "F.Mask")
       (net 81 "/SDA"))
-    (model "${KISYS3DMOD}/Resistors_SMD.3dshapes/R_0603.wrl"
+    (model "${KICAD6_3DMODEL_DIR}/Resistor_SMD.3dshapes/R_0603_1608Metric.wrl"
       (offset (xyz 0 0 0))
       (scale (xyz 1 1 1))
@@
     (pad "2" smd rect locked (at 0.75 0 270) (size 0.5 0.9) (layers "F.Cu" "F.Paste" "F.Mask")
       (net 80 "/SCL"))
-    (model "${KISYS3DMOD}/Resistors_SMD.3dshapes/R_0603.wrl"
+    (model "${KICAD6_3DMODEL_DIR}/Resistor_SMD.3dshapes/R_0603_1608Metric.wrl"
       (offset (xyz 0 0 0))
       (scale (xyz 1 1 1))
@@
     (pad "2" smd rect locked (at 0.75 0 270) (size 0.5 0.9) (layers "F.Cu" "F.Paste" "F.Mask")
       (net 23 "Net-(JP1-Pad2)"))
-    (model "${KISYS3DMOD}/Resistors_SMD.3dshapes/R_0603.wrl"
+    (model "${KICAD6_3DMODEL_DIR}/Resistor_SMD.3dshapes/R_0603_1608Metric.wrl"
       (offset (xyz 0 0 0))
       (scale (xyz 1 1 1))
@@
     (pad "2" smd rect locked (at 0.75 0 90) (size 0.5 0.9) (layers "F.Cu" "F.Paste" "F.Mask")
       (net 24 "Net-(JP2-Pad2)"))
-    (model "${KISYS3DMOD}/Resistors_SMD.3dshapes/R_0603.wrl"
+    (model "${KICAD6_3DMODEL_DIR}/Resistor_SMD.3dshapes/R_0603_1608Metric.wrl"
       (offset (xyz 0 0 0))
       (scale (xyz 1 1 1))
@@
     (pad "2" smd rect locked (at 0.75 0 90) (size 0.5 0.9) (layers "F.Cu" "F.Paste" "F.Mask")
       (net 102 "Net-(R8-Pad2)"))
-    (model "${KISYS3DMOD}/Resistors_SMD.3dshapes/R_0603.wrl"
+    (model "${KICAD6_3DMODEL_DIR}/Resistor_SMD.3dshapes/R_0603_1608Metric.wrl"
       (offset (xyz 0 0 0))
       (scale (xyz 1 1 1))
@@
     (pad "2" smd rect locked (at 0.75 0 270) (size 0.5 0.9) (layers "F.Cu" "F.Paste" "F.Mask")
       (net 25 "Net-(JP3-Pad2)"))
-    (model "${KISYS3DMOD}/Resistors_SMD.3dshapes/R_0603.wrl"
-      (offset (xyz 0 0 0))
-      (scale (xyz 1 1 1))
-      (rotate (xyz 0 0 0))
-    )
-  )
-  (footprint "Connectors_Terminal_Blocks:TerminalBlock_Pheonix_MPT-2.54mm_2pol" (layer "F.Cu")
+    (model "${KICAD6_3DMODEL_DIR}/Resistor_SMD.3dshapes/R_0603_1608Metric.wrl"
+      (offset (xyz 0 0 0))
+      (scale (xyz 1 1 1))
+      (rotate (xyz 0 0 0))
+    )
+  )
+  (footprint "Connectors_Terminal_Blocks:TerminalBlock_Phoenix_MPT-2.54mm_2pol" (layer "F.Cu")
     (at 133.35 135.89)
     (descr "2-way 2.54mm pitch terminal block, Phoenix MPT series")
@@
     (pad "2" thru_hole oval locked (at 2.54 0) (size 1.99898 1.99898) (drill 1.09728) (layers *.Cu *.Mask)
       (net 7 "GND"))
-    (model "Terminal_Blocks.3dshapes/TerminalBlock_Pheonix_MPT-2.54mm_2pol.wrl"
+    (model "${KICAD6_3DMODEL_DIR}/TerminalBlock_Phoenix.3dshapes/TerminalBlock_Phoenix_MPT-0,5-2-2.54_1x02_P2.54mm_Horizontal.wrl"
       (offset (xyz 1.269999981 0 0))
       (scale (xyz 1 1 1))
@@
     )
   )
-  (footprint "Connectors_Terminal_Blocks:TerminalBlock_Pheonix_MPT-2.54mm_2pol" (layer "F.Cu")
+  (footprint "Connectors_Terminal_Blocks:TerminalBlock_Phoenix_MPT-2.54mm_2pol" (layer "F.Cu")
     (at 146.05 135.89)
     (descr "2-way 2.54mm pitch terminal block, Phoenix MPT series")
@@
     (pad "2" thru_hole oval locked (at 2.54 0) (size 1.99898 1.99898) (drill 1.09728) (layers *.Cu *.Mask)
       (net 7 "GND"))
-    (model "Terminal_Blocks.3dshapes/TerminalBlock_Pheonix_MPT-2.54mm_2pol.wrl"
+    (model "${KICAD6_3DMODEL_DIR}/TerminalBlock_Phoenix.3dshapes/TerminalBlock_Phoenix_MPT-0,5-2-2.54_1x02_P2.54mm_Horizontal.wrl"
       (offset (xyz 1.269999981 0 0))
       (scale (xyz 1 1 1))
@@
     (pad "8" smd rect locked (at 2.7 -1.905) (size 1.55 0.6) (layers "F.Cu" "F.Paste" "F.Mask")
       (net 1 "+3V3"))
-    (model "${KISYS3DMOD}/Housings_SOIC.3dshapes/SOIC-8_3.9x4.9mm_Pitch1.27mm.wrl"
-      (offset (xyz 0 0 0))
-      (scale (xyz 1 1 1))
+    (model "${KICAD6_3DMODEL_DIR}/Package_SO.3dshapes/SOIC-8_3.9x4.9mm_P1.27mm.wrl"
+      (offset (xyz 0 0 0))
+      (scale (xyz 1 1 1))
