File: FRED/FRED.kicad_sch (KiCad schematic)
At the start: 11 parts, among them U101 LM555xMM

Commit message: Design a FRED.
Parts:
- removed TP101: Track, Connector_Wire:SolderWire-0.1sqmm_1x02_P3.6mm_D0.4mm_OD1mm, symbol Connector:TestPoint_2Pole
- added TP101: RightTrack, Pads:Track Pickup Pad, symbol Connector:TestPoint
- added TP104: Left Track, Pads:Track Pickup Pad, symbol Connector:TestPoint
- C101: footprint Capacitor_SMD:CP_Elec_6.3x7.7 -> Capacitor_Tantalum_SMD:CP_EIA-7343-43_Kemet-X; Mouser Part Nunber 710-865080445010 -> 581-TPME107K025R0045
- TP103: value + LED - -> + -
Connections:
- net at D101.3: now also TP101.1
- net at D101.4: now also TP104.1
Changed lines of the file:
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@@
     (pin "1")
   )
-  (symbol (lib_id "Connector:TestPoint_2Pole") (at 64.135 75.565 0) (unit 1)
-    (in_bom yes) (on_board yes) (fields_autoplaced)
-    (property "Reference" "TP101" (id 0) (at 64.135 69.85 0))
-    (property "Value" "Track" (id 1) (at 64.135 72.39 0))
-    (property "Footprint" "Connector_Wire:SolderWire-0.1sqmm_1x02_P3.6mm_D0.4mm_OD1mm" (id 2) (at 64.135 75.565 0)
+  (symbol (lib_id "Connector:TestPoint") (at 59.055 75.565 0) (unit 1)
+    (in_bom yes) (on_board yes) (fields_autoplaced)
+    (property "Reference" "TP101" (id 0) (at 60.96 70.9929 0)
+      (effects (font (size 1.27 1.27)) (justify left))
+    )
+    (property "Value" "RightTrack" (id 1) (at 60.96 73.5329 0)
+      (effects (font (size 1.27 1.27)) (justify left))
+    )
+    (property "Footprint" "Pads:Track Pickup Pad" (id 2) (at 64.135 75.565 0)
       (effects (font (size 1.27 1.27)) hide)
     )
@@
     )
     (pin "1")
-    (pin "2")
   )
   (symbol (lib_id "Device:C_Polarized_Small_US") (at 81.28 59.055 0) (unit 1)
@@
       (effects (font (size 1.27 1.27)) (justify left))
     )
-    (property "Footprint" "Capacitor_SMD:CP_Elec_6.3x7.7" (id 2) (at 81.28 59.055 0)
+    (property "Footprint" "Capacitor_Tantalum_SMD:CP_EIA-7343-43_Kemet-X" (id 2) (at 81.28 59.055 0)
       (effects (font (size 1.27 1.27)) hide)
     )
@@
       (effects (font (size 1.27 1.27)) hide)
     )
-    (property "Mouser Part Nunber" "710-865080445010" (id 4) (at 81.28 59.055 0)
+    (property "Mouser Part Nunber" "581-TPME107K025R0045" (id 4) (at 81.28 59.055 0)
       (effects (font (size 1.27 1.27)) hide)
     )
@@
     (in_bom yes) (on_board yes) (fields_autoplaced)
     (property "Reference" "TP103" (id 0) (at 202.565 53.34 0))
-    (property "Value" "+ LED -" (id 1) (at 202.565 55.88 0))
+    (property "Value" "+  -" (id 1) (at 202.565 55.88 0))
     (property "Footprint" "Pads:SolderPads_1x2_1.2mm" (id 2) (at 202.565 59.055 0)
       (effects (font (size 1.27 1.27)) hide)
@@
     (pin "2")
   )
+  (symbol (lib_id "Connector:TestPoint") (at 69.215 75.565 0) (unit 1)
+    (in_bom yes) (on_board yes) (fields_autoplaced)
+    (property "Reference" "TP104" (id 0) (at 71.12 70.9929 0)
+      (effects (font (size 1.27 1.27)) (justify left))
+    )
+    (property "Value" "Left Track" (id 1) (at 71.12 73.5329 0)
+      (effects (font (size 1.27 1.27)) (justify left))
+    )
+    (property "Footprint" "Pads:Track Pickup Pad" (id 2) (at 74.295 75.565 0)
+      (effects (font (size 1.27 1.27)) hide)
+    )
+    (property "Datasheet" "~" (id 3) (at 74.295 75.565 0)
+      (effects (font (size 1.27 1.27)) hide)
+    )
+    (pin "1")
+  )
   (sheet_instances
     (path "/" (page "1"))
@@
     )
     (path "/62656f08-78ab-42c1-9b0e-309545d0a6fa"
-      (reference "C101") (unit 1) (value "100uf 25V") (footprint "Capacitor_SMD:CP_Elec_6.3x7.7")
+      (reference "C101") (unit 1) (value "100uf 25V") (footprint "Capacitor_Tantalum_SMD:CP_EIA-7343-43_Kemet-X")
     )
     (path "/8b764051-f191-46fd-bc3d-0b22f8af5e5b"
@@
       (reference "R102") (unit 1) (value "1K5") (footprint "Resistor_SMD:R_0402_1005Metric")
     )
-    (path "/365a220b-3fe6-4526-9a8e-a544812c602b"
-      (reference "TP101") (unit 1) (value "Track") (footprint "Connector_Wire:SolderWire-0.1sqmm_1x02_P3.6mm_D0.4mm_OD1mm")
+    (path "/3f78aded-4814-46f6-afd1-cccfbbf3bf75"
+      (reference "TP101") (unit 1) (value "RightTrack") (footprint "Pads:Track Pickup Pad")
     )
     (path "/01396b2c-09c2-4a0f-a22f-2fa71038a517"
@@
     )
     (path "/9c301b9e-eebf-4c0a-817f-487b8ae3089b"
-      (reference "TP103") (unit 1) (value "+ LED -") (footprint "Pads:SolderPads_1x2_1.2mm")
+      (reference "TP103") (unit 1) (value "+  -") (footprint "Pads:SolderPads_1x2_1.2mm")
+    )
+    (path "/f3b6f614-a805-4027-a398-1285c6ca597c"
+      (reference "TP104") (unit 1) (value "Left Track") (footprint "Pads:Track Pickup Pad")
     )
     (path "/6c9b793c-e74d-4754-a2c0-901e73b26f1c"

Commit message: Part number updates.
Parts:
- C101: Mouser Part Number (none) -> 581-TPME107K025R0045; Mouser Part Nunber 581-TPME107K025R0045 -> (none)
- C102: Mouser Part Number 80-C0402C103K3R7867 -> 603-CC402JRX7R8BB103
- C103: Mouser Part Number 603-AC402KRX5R5BB105 -> 603-CC402KRX5R6BB105
Changed lines of the file:
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@@
       (effects (font (size 1.27 1.27)) hide)
     )
-    (property "Mouser Part Nunber" "581-TPME107K025R0045" (id 4) (at 81.28 59.055 0)
+    (property "Mouser Part Number" "581-TPME107K025R0045" (id 4) (at 81.28 59.055 0)
       (effects (font (size 1.27 1.27)) hide)
     )
@@
       (effects (font (size 1.27 1.27)) hide)
     )
-    (property "Mouser Part Number" "603-AC402KRX5R5BB105" (id 4) (at 156.21 92.075 0)
+    (property "Mouser Part Number" "603-CC402KRX5R6BB105" (id 4) (at 156.21 92.075 0)
       (effects (font (size 1.27 1.27)) hide)
     )
@@
       (effects (font (size 1.27 1.27)) hide)
     )
-    (property "Mouser Part Number" "80-C0402C103K3R7867" (id 4) (at 111.125 87.63 0)
+    (property "Mouser Part Number" "603-CC402JRX7R8BB103" (id 4) (at 111.125 87.63 0)
       (effects (font (size 1.27 1.27)) hide)
     )

Commit message: Tweaks to FRED.
Parts:
- C101: footprint Capacitor_Tantalum_SMD:CP_EIA-7343-43_Kemet-X -> Capacitor_Tantalum_SMD:CP_EIA-7361-438_AVX-U; Mouser Part Number 581-TPME107K025R0045 -> 581-TRJU107K025RRJV
Changed lines of the file:
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@@
       (effects (font (size 1.27 1.27)) (justify left))
     )
-    (property "Footprint" "Capacitor_Tantalum_SMD:CP_EIA-7343-43_Kemet-X" (id 2) (at 81.28 59.055 0)
+    (property "Footprint" "Capacitor_Tantalum_SMD:CP_EIA-7361-438_AVX-U" (id 2) (at 81.28 59.055 0)
       (effects (font (size 1.27 1.27)) hide)
     )
@@
       (effects (font (size 1.27 1.27)) hide)
     )
-    (property "Mouser Part Number" "581-TPME107K025R0045" (id 4) (at 81.28 59.055 0)
+    (property "Mouser Part Number" "581-TRJU107K025RRJV" (id 4) (at 81.28 59.055 0)
       (effects (font (size 1.27 1.27)) hide)
     )
@@
     )
     (path "/62656f08-78ab-42c1-9b0e-309545d0a6fa"
-      (reference "C101") (unit 1) (value "100uf 25V") (footprint "Capacitor_Tantalum_SMD:CP_EIA-7343-43_Kemet-X")
+      (reference "C101") (unit 1) (value "100uf 25V") (footprint "Capacitor_Tantalum_SMD:CP_EIA-7361-438_AVX-U")
     )
     (path "/8b764051-f191-46fd-bc3d-0b22f8af5e5b"
